File: Xaar128-Driver/reset_circuit.kicad_sch (KiCad schematic)
At the start: 44 parts, among them Q1 DMN2075U, Q2 DMN2075U, Q3 DMN2075U, Q7 DMG2305UX, U1 6N135, U2 6N135, U3 74HC173

Commit message: 5v monitoring
Parts:
- removed R15: 10k, symbol Device:R
Other:
- moved on the sheet: C7, D1, D2, D4, D5, JP4, JP5, JP6, JP7, Q1, Q2, Q3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

Commit message: some component selections, fix wrong mcu
Parts:
- C7: value 100n -> 100n >16V Cer; footprint (none) -> Capacitor_SMD:C_0603_1608Metric_Pad1.08x0.95mm_HandSolder; Supplier (none) -> Elektroplatz
- JP4: value RST_36V -> Jumper_3_Bridged12; footprint (none) -> Connector_PinHeader_2.54mm:PinHeader_1x03_P2.54mm_Vertical; Funktion (none) -> Disable Reset on 36V loss
- JP5: value RST_VPP -> Jumper_3_Bridged12; footprint (none) -> Connector_PinHeader_2.54mm:PinHeader_1x03_P2.54mm_Vertical; Funktion (none) -> Disable Reset on VPP loss
- JP6: value RST_MCU -> Jumper_3_Bridged12; footprint (none) -> Connector_PinHeader_2.54mm:PinHeader_1x03_P2.54mm_Vertical; Funktion (none) -> Disable Reset on MCU
- JP7: value RST_nFAULT -> Jumper_3_Bridged12; footprint (none) -> Connector_PinHeader_2.54mm:PinHeader_1x03_P2.54mm_Vertical; Funktion (none) -> Disable Reset on nFault
- Q1, Q2, Q3: RSBestNr (none) -> 751-4143; Supplier (none) -> RS
- Q7: RSBestNr (none) -> 827-0452; Supplier (none) -> RS
- TP1: value Q1_Gate -> TestPoint; footprint (none) -> TestPoint:TestPoint_Pad_D1.5mm; Funktion (none) -> Q1_Gate; Supplier (none) -> None
- TP2: value Q2_Gate -> TestPoint; footprint (none) -> TestPoint:TestPoint_Pad_D1.5mm; Funktion (none) -> Q2_Gate; Supplier (none) -> None
- TP3: value nRESET_FAULT -> TestPoint; footprint (none) -> TestPoint:TestPoint_Pad_D1.5mm; Funktion (none) -> nRESET_FAULT; Supplier (none) -> None
- TP4: value nRESET -> TestPoint; footprint (none) -> TestPoint:TestPoint_Pad_D1.5mm; Funktion (none) -> nRESET; Supplier (none) -> None
- U1, U2: RSBestNr (none) -> 691-2316; Supplier (none) -> RS

Commit message: assign footprints
Parts:
- removed D1: 27V, symbol Device:D_Zener
- removed D2: 10V, symbol Device:D_Zener
- added D1: BZX84C10LT1G 10V, Package_TO_SOT_SMD:SOT-23, symbol Diode:BZX84Cxx
- added D6: BZX84C27LT1G 27V, Package_TO_SOT_SMD:SOT-23, symbol Diode:BZX84Cxx
- D4, D5: footprint (none) -> LED_THT:LED_D5.0mm; Supplier (none) -> Elektroplatz
- JP4, JP5, JP6, JP7: Supplier (none) -> Elektroplatz
- R10, R3, R5: footprint (none) -> Resistor_SMD:R_0603_1608Metric_Pad0.98x0.95mm_HandSolder; RSBestNr (none) -> 678-9875; Supplier (none) -> RS
- R11: value 2k -> 2k > 700mW
- R13, R15, R16, R17: footprint (none) -> Resistor_SMD:R_0603_1608Metric_Pad0.98x0.95mm_HandSolder; Supplier (none) -> Elektroplatz
- R14, R17: footprint (none) -> Resistor_SMD:R_0603_1608Metric_Pad0.98x0.95mm_HandSolder; RSBestNr (none) -> 678-9673; Supplier (none) -> RS
- R8: value 5.1k -> 5.1k >300mW
- U3: footprint (none) -> Package_SO:SO-16_3.9x9.9mm_P1.27mm; RSBestNr (none) -> 483-6443; Supplier (none) -> RS
Connections:
- net at R1.2, R4.1: now also D6.3 (K)
- net at R2.1, R5.1: now also D6.1 (A)
- net at R10.1, R9.1: now also D1.1 (A)
- net at R6.2, R7.1: now also D1.3 (K)

Commit message: select remaining components, nucleo footprint
Parts:
- C7: value 100n >16V Cer -> (none)
- R1: footprint (none) -> Resistor_SMD:R_0603_1608Metric_Pad0.98x0.95mm_HandSolder; RSBestNr (none) -> 198-5480; Supplier (none) -> RS
- R11: footprint (none) -> Resistor_SMD:R_2010_5025Metric_Pad1.40x2.65mm_HandSolder; RSBestNr (none) -> 186-6957; Supplier (none) -> RS
- R12: footprint (none) -> Resistor_SMD:R_0603_1608Metric_Pad0.98x0.95mm_HandSolder; Supplier (none) -> Elektroplatz
- R2, R9: footprint (none) -> Resistor_SMD:R_0603_1608Metric_Pad0.98x0.95mm_HandSolder; RSBestNr (none) -> 242-4070; Supplier (none) -> RS
- R4: value 32k -> 31.5k; footprint (none) -> Resistor_THT:R_Axial_DIN0207_L6.3mm_D2.5mm_P7.62mm_Horizontal; Supplier (none) -> Elektroplatz
- R6: footprint (none) -> Resistor_SMD:R_0603_1608Metric_Pad0.98x0.95mm_HandSolder; RSBestNr (none) -> 198-5552; Supplier (none) -> RS
- R7: footprint (none) -> Resistor_SMD:R_0603_1608Metric_Pad0.98x0.95mm_HandSolder; RSBestNr (none) -> 566-367; Supplier (none) -> RS
- R8: footprint (none) -> Resistor_SMD:R_0805_2012Metric_Pad1.20x1.40mm_HandSolder; RSBestNr (none) -> 721-7804; Supplier (none) -> RS
Changed lines of the file:
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@@
       (effects (font (size 1.27 1.27)) (justify left))
     )
-    (property "Footprint" "" (at 35.052 48.26 90)
+    (property "Footprint" "Resistor_SMD:R_0603_1608Metric_Pad0.98x0.95mm_HandSolder" (at 35.052 48.26 90)
       (effects (font (size 1.27 1.27)) hide)
     )
@@
       (effects (font (size 1.27 1.27)) hide)
     )
-    (property "RSBestNr" "" (at 36.83 48.26 0)
-      (effects (font (size 1.27 1.27)) hide)
-    )
-    (property "Supplier" "" (at 36.83 48.26 0)
+    (property "RSBestNr" "198-5480" (at 36.83 48.26 0)
+      (effects (font (size 1.27 1.27)) hide)
+    )
+    (property "Supplier" "RS" (at 36.83 48.26 0)
       (effects (font (size 1.27 1.27)) hide)
     )
@@
       (effects (font (size 1.27 1.27)) (justify left))
     )
-    (property "Footprint" "" (at 46.482 80.01 90)
+    (property "Footprint" "Resistor_SMD:R_0603_1608Metric_Pad0.98x0.95mm_HandSolder" (at 46.482 80.01 90)
       (effects (font (size 1.27 1.27)) hide)
     )
@@
       (effects (font (size 1.27 1.27)) hide)
     )
-    (property "RSBestNr" "" (at 48.26 80.01 0)
-      (effects (font (size 1.27 1.27)) hide)
-    )
-    (property "Supplier" "" (at 48.26 80.01 0)
+    (property "RSBestNr" "242-4070" (at 48.26 80.01 0)
+      (effects (font (size 1.27 1.27)) hide)
+    )
+    (property "Supplier" "RS" (at 48.26 80.01 0)
       (effects (font (size 1.27 1.27)) hide)
     )
@@
       (effects (font (size 1.27 1.27)) (justify left))
     )
-    (property "Footprint" "" (at 46.482 133.35 90)
+    (property "Footprint" "Resistor_SMD:R_0603_1608Metric_Pad0.98x0.95mm_HandSolder" (at 46.482 133.35 90)
       (effects (font (size 1.27 1.27)) hide)
     )
@@
       (effects (font (size 1.27 1.27)) hide)
     )
-    (property "RSBestNr" "" (at 48.26 133.35 0)
-      (effects (font (size 1.27 1.27)) hide)
-    )
-    (property "Supplier" "" (at 48.26 133.35 0)
+    (property "RSBestNr" "242-4070" (at 48.26 133.35 0)
+      (effects (font (size 1.27 1.27)) hide)
+    )
+    (property "Supplier" "RS" (at 48.26 133.35 0)
       (effects (font (size 1.27 1.27)) hide)
     )
@@
       (effects (font (size 1.27 1.27)))
     )
-    (property "Footprint" "" (at 66.04 98.298 90)
+    (property "Footprint" "Resistor_SMD:R_2010_5025Metric_Pad1.40x2.65mm_HandSolder" (at 66.04 98.298 90)
       (effects (font (size 1.27 1.27)) hide)
     )
@@
       (effects (font (size 1.27 1.27)) hide)
     )
-    (property "RSBestNr" "" (at 66.04 96.52 0)
-      (effects (font (size 1.27 1.27)) hide)
-    )
-    (property "Supplier" "" (at 66.04 96.52 0)
+    (property "RSBestNr" "186-6957" (at 66.04 96.52 0)
+      (effects (font (size 1.27 1.27)) hide)
+    )
+    (property "Supplier" "RS" (at 66.04 96.52 0)
       (effects (font (size 1.27 1.27)) hide)
     )
@@
       (effects (font (size 1.27 1.27)))
     )
-    (property "Value" "100n >16V Cer" (at 220.98 21.59 90)
+    (property "Value" "  " (at 220.98 21.59 90)
       (effects (font (size 1.27 1.27)))
     )
@@
       (effects (font (size 1.27 1.27)) (justify left))
     )
-    (property "Footprint" "" (at 35.052 101.6 90)
+    (property "Footprint" "Resistor_SMD:R_0603_1608Metric_Pad0.98x0.95mm_HandSolder" (at 35.052 101.6 90)
       (effects (font (size 1.27 1.27)) hide)
     )
@@
       (effects (font (size 1.27 1.27)) hide)
     )
-    (property "RSBestNr" "" (at 36.83 101.6 0)
-      (effects (font (size 1.27 1.27)) hide)
-    )
-    (property "Supplier" "" (at 36.83 101.6 0)
+    (property "RSBestNr" "198-5552" (at 36.83 101.6 0)
+      (effects (font (size 1.27 1.27)) hide)
+    )
+    (property "Supplier" "RS" (at 36.83 101.6 0)
       (effects (font (size 1.27 1.27)) hide)
     )
@@
       (effects (font (size 1.27 1.27)) (justify left))
     )
-    (property "Value" "32k" (at 39.37 76.2 0)
-      (effects (font (size 1.27 1.27)) (justify left))
-    )
-    (property "Footprint" "" (at 35.052 74.93 90)
+    (property "Value" "31.5k" (at 39.37 76.2 0)
+      (effects (font (size 1.27 1.27)) (justify left))
+    )
+    (property "Footprint" "Resistor_THT:R_Axial_DIN0207_L6.3mm_D2.5mm_P7.62mm_Horizontal" (at 35.052 74.93 90)
       (effects (font (size 1.27 1.27)) hide)
     )
@@
       (effects (font (size 1.27 1.27)) hide)
     )
-    (property "Supplier" "" (at 36.83 74.93 0)
+    (property "Supplier" "Elektroplatz" (at 36.83 74.93 0)
       (effects (font (size 1.27 1.27)) hide)
     )
@@
       (effects (font (size 1.27 1.27)) (justify left))
     )
-    (property "Footprint" "" (at 35.052 127 90)
+    (property "Footprint" "Resistor_SMD:R_0603_1608Metric_Pad0.98x0.95mm_HandSolder" (at 35.052 127 90)
       (effects (font (size 1.27 1.27)) hide)
     )
@@
       (effects (font (size 1.27 1.27)) hide)
     )
-    (property "RSBestNr" "" (at 36.83 127 0)
-      (effects (font (size 1.27 1.27)) hide)
-    )
-    (property "Supplier" "" (at 36.83 127 0)
+    (property "RSBestNr" "566-367" (at 36.83 127 0)
+      (effects (font (size 1.27 1.27)) hide)
+    )
+    (property "Supplier" "RS" (at 36.83 127 0)
       (effects (font (size 1.27 1.27)) hide)
     )
@@
       (effects (font (size 1.27 1.27)))
     )
-    (property "Footprint" "" (at 66.04 44.958 90)
+    (property "Footprint" "Resistor_SMD:R_0805_2012Metric_Pad1.20x1.40mm_HandSolder" (at 66.04 44.958 90)
       (effects (font (size 1.27 1.27)) hide)
     )
@@
       (effects (font (size 1.27 1.27)) hide)
     )
-    (property "RSBestNr" "" (at 66.04 43.18 0)
-      (effects (font (size 1.27 1.27)) hide)
-    )
-    (property "Supplier" "" (at 66.04 43.18 0)
+    (property "RSBestNr" "721-7804" (at 66.04 43.18 0)
+      (effects (font (size 1.27 1.27)) hide)
+    )
+    (property "Supplier" "RS" (at 66.04 43.18 0)
       (effects (font (size 1.27 1.27)) hide)
     )
@@
       (effects (font (size 1.27 1.27)) (justify left))
     )
-    (property "Footprint" "" (at 132.842 30.48 90)
+    (property "Footprint" "Resistor_SMD:R_0603_1608Metric_Pad0.98x0.95mm_HandSolder" (at 132.842 30.48 90)
       (effects (font (size 1.27 1.27)) hide)
     )
@@
       (effects (font (size 1.27 1.27)) hide)
     )
-    (property "Supplier" "" (at 134.62 30.48 0)
-      (effects (font (size 1.27 1.27)) hide)
-    )
+    (property "Supplier" "Elektroplatz" (at 134.62 30.48 0)
+      (effects (font (size 1.27 1.27)) hide)
+    )

Commit message: xaar driver: some routed islands
Parts:
- added NT3: NetTie_2, NetTie:NetTie-2_SMD_Pad0.5mm, symbol Device:NetTie_2
Connections:
- net +36V: now also NT3.1; no longer R1.1, R8.1
- new net: NT3.2, R1.1, R8.1
Changed lines of the file:
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@@
   (junction (at 134.62 50.8) (diameter 0) (color 0 0 0 0)
   )
+  (junction (at 36.83 43.18) (diameter 0) (color 0 0 0 0)
+  )
   (junction (at 165.1 26.67) (diameter 0) (color 0 0 0 0)
   )
@@
   )
   (junction (at 36.83 58.42) (diameter 0) (color 0 0 0 0)
-  )
-  (junction (at 36.83 43.18) (diameter 0) (color 0 0 0 0)
   )
   (junction (at 36.83 87.63) (diameter 0) (color 0 0 0 0)
@@
     (stroke (width 0) (type default))
   )
-  (wire (pts (xy 21.59 43.18) (xy 36.83 43.18))
-    (stroke (width 0) (type default))
-  )
   (wire (pts (xy 22.86 96.52) (xy 36.83 96.52))
     (stroke (width 0) (type default))
@@
     (stroke (width 0) (type default))
   )
+  (wire (pts (xy 31.75 43.18) (xy 36.83 43.18))
+    (stroke (width 0) (type default))
+  )
   (wire (pts (xy 134.62 101.6) (xy 134.62 104.14))
     (stroke (width 0) (type default))
@@
   )
   (wire (pts (xy 105.41 104.14) (xy 134.62 104.14))
+    (stroke (width 0) (type default))
+  )
+  (wire (pts (xy 21.59 43.18) (xy 26.67 43.18))
     (stroke (width 0) (type default))
   )
@@
     (effects (font (size 1.27 1.27)) (justify left bottom))
     (property "Netclass" "HV" (at 34.29 118.6815 90)
+      (effects (font (size 1.27 1.27) italic) (justify left))
+    )
+  )
+  (netclass_flag "" (length 2.54) (shape round) (at 48.26 43.18 180) (fields_autoplaced)
+    (effects (font (size 1.27 1.27)) (justify right bottom))
+    (property "Netclass" "HV" (at 48.9585 45.72 0)
       (effects (font (size 1.27 1.27) italic) (justify left))
     )
@@
         )
       )
+    )
+  )
+  (symbol (lib_id "Device:NetTie_2") (at 29.21 43.18 0) (unit 1)
+    (in_bom no) (on_board yes) (dnp no) (fields_autoplaced)
+    (property "Reference" "NT3" (at 29.21 38.1 0)
+      (effects (font (size 1.27 1.27)))
+    )
+    (property "Value" "NetTie_2" (at 29.21 40.64 0)
+      (effects (font (size 1.27 1.27)))
+    )
+    (property "Footprint" "NetTie:NetTie-2_SMD_Pad0.5mm" (at 29.21 43.18 0)
+      (effects (font (size 1.27 1.27)) hide)
+    )
+    (property "Datasheet" "~" (at 29.21 43.18 0)
+      (effects (font (size 1.27 1.27)) hide)
+    )
+    (property "Supplier" "None" (at 29.21 43.18 0)
+      (effects (font (size 1.27 1.27)) hide)
+    )
+    (pin "1")
+    (pin "2")
+    (instances
+      (project "Xaar128-Driver"
+        (path "/f0c82013-03f9-4093-aa02-30b89fd69529/48b639c9-d588-4ad3-b95b-9aa4a2d6905e"
+          (reference "NT3") (unit 1)
+        )
+        (path "/f0c82013-03f9-4093-aa02-30b89fd69529/7aab5eaf-cd9d-4ebb-9d08-de265e07412e"
+          (reference "NT4") (unit 1)
+        )
+      )

Commit message: more routing
Parts:
- removed R17: 100k, Resistor_SMD:R_0603_1608Metric_Pad0.98x0.95mm_HandSolder, symbol Device:R
Changed lines of the file:
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@@
   (junction (at 36.83 43.18) (diameter 0) (color 0 0 0 0)
   )
-  (junction (at 165.1 26.67) (diameter 0) (color 0 0 0 0)
-  )
   (junction (at 144.78 63.5) (diameter 0) (color 0 0 0 0)
   )
@@
   )
   (junction (at 134.62 39.37) (diameter 0) (color 0 0 0 0)
-  )
-  (junction (at 161.29 39.37) (diameter 0) (color 0 0 0 0)
   )
   (junction (at 186.69 121.92) (diameter 0) (color 0 0 0 0)
@@
     (stroke (width 0) (type default))
   )
-  (wire (pts (xy 161.29 29.21) (xy 161.29 26.67))
-    (stroke (width 0) (type default))
-  )
   (wire (pts (xy 105.41 101.6) (xy 121.92 101.6))
     (stroke (width 0) (type default))
@@
     (stroke (width 0) (type default))
   )
-  (wire (pts (xy 161.29 36.83) (xy 161.29 39.37))
-    (stroke (width 0) (type default))
-  )
   (wire (pts (xy 236.22 54.61) (xy 236.22 49.53))
     (stroke (width 0) (type default))
@@
   )
   (wire (pts (xy 236.22 62.23) (xy 236.22 72.39))
-    (stroke (width 0) (type default))
-  )
-  (wire (pts (xy 161.29 26.67) (xy 165.1 26.67))
     (stroke (width 0) (type default))
   )
@@
         )
       )
-    )
-  )
-  (symbol (lib_id "Device:R") (at 161.29 33.02 180) (unit 1)
-    (in_bom yes) (on_board yes) (dnp yes)
-    (property "Reference" "R17" (at 160.02 31.75 0)
-      (effects (font (size 1.27 1.27)) (justify left))
-    )
-    (property "Value" "100k" (at 160.02 34.29 0)
-      (effects (font (size 1.27 1.27)) (justify left))
-    )
-    (property "Footprint" "Resistor_SMD:R_0603_1608Metric_Pad0.98x0.95mm_HandSolder" (at 163.068 33.02 90)
-      (effects (font (size 1.27 1.27)) hide)
-    )
-    (property "Datasheet" "~" (at 161.29 33.02 0)
-      (effects (font (size 1.27 1.27)) hide)
-    )
-    (property "RSBestNr" "678-9673" (at 161.29 33.02 0)
-      (effects (font (size 1.27 1.27)) hide)
-    )
-    (property "Supplier" "RS" (at 161.29 33.02 0)
-      (effects (font (size 1.27 1.27)) hide)
-    )
-    (pin "1")
-    (pin "2")
-    (instances
-      (project "Xaar128-Driver"
-        (path "/f0c82013-03f9-4093-aa02-30b89fd69529"
-          (reference "R17") (unit 1)
-        )
-        (path "/f0c82013-03f9-4093-aa02-30b89fd69529/7aab5eaf-cd9d-4ebb-9d08-de265e07412e"
-          (reference "R48") (unit 1)
-        )
-      )

Commit message: more routing
Connections:
- net GND: now also JP6.3 (B), Q3.2 (S); no longer JP7.3 (B), Q3.2 (S)
- net nRESET_FAULT: now also JP7.2 (C); no longer JP4.2 (C)
- net at JP5.3 (B), U2.5: now also JP4.2 (C); no longer JP6.2 (C)
- net at JP4.3 (B), U1.5: now also JP6.2 (C); no longer JP5.2 (C)
- new net: JP5.2 (C), JP7.3 (B), Q3.2 (S)
Other:
- moved on the sheet: D1, D4, D5, D6, JP4, JP5, JP6, NT3, Q1, Q2, Q3, R1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

Commit message: almost
Parts:
- R4: value 31.5k -> 31.6k; footprint Resistor_THT:R_Axial_DIN0207_L6.3mm_D2.5mm_P7.62mm_Horizontal -> Resistor_SMD:R_0603_1608Metric_Pad0.98x0.95mm_HandSolder; RSBestNr (none) -> 708-8877; Supplier Elektroplatz -> RS
Changed lines of the file:
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@@
       (effects (font (size 1.27 1.27)) (justify left))
     )
-    (property "Value" "31.5k" (at 39.37 160.02 0)
+    (property "Value" "31.6k" (at 39.37 160.02 0)
       (effects (font (size 1.27 1.27)) (justify left))
     )
-    (property "Footprint" "Resistor_THT:R_Axial_DIN0207_L6.3mm_D2.5mm_P7.62mm_Horizontal" (at 35.052 158.75 90)
+    (property "Footprint" "Resistor_SMD:R_0603_1608Metric_Pad0.98x0.95mm_HandSolder" (at 35.052 158.75 90)
       (effects (font (size 1.27 1.27)) hide)
     )
@@
       (effects (font (size 1.27 1.27)) hide)
     )
-    (property "RSBestNr" "" (at 36.83 158.75 0)
+    (property "RSBestNr" "708-8877" (at 36.83 158.75 0)
       (effects (font (size 1.27 1.27)) hide)
     )
-    (property "Supplier" "Elektroplatz" (at 36.83 158.75 0)
+    (property "Supplier" "RS" (at 36.83 158.75 0)
       (effects (font (size 1.27 1.27)) hide)
     )
