File: Xaar128-Driver/reset_circuit.kicad_sch (KiCad schematic)
At the start: 43 parts, among them Q1 DMN2075U, Q2 DMN2075U, Q3 DMN2075U, Q7 DMG2305UX, U1 6N135, U2 6N135, U3 74HC173

Commit message: drc & plots done
Parts:
- D4, D5: footprint LED_THT:LED_D5.0mm -> Custom_LED_THT:LED_D5.0mm
- TP1, TP2, TP3, TP4: footprint TestPoint:TestPoint_Pad_D1.5mm -> Xaar-Driver:TestPoint_Pad_D1.5mm
Changed lines of the file:
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@@
       (effects (font (size 1.27 1.27)) (justify right))
     )
-    (property "Footprint" "TestPoint:TestPoint_Pad_D1.5mm" (at 247.65 38.1 0)
+    (property "Footprint" "Xaar-Driver:TestPoint_Pad_D1.5mm" (at 247.65 38.1 0)
       (effects (font (size 1.27 1.27)) hide)
     )
@@
       (effects (font (size 1.27 1.27)) (justify right))
     )
-    (property "Footprint" "LED_THT:LED_D5.0mm" (at 90.17 83.82 0)
+    (property "Footprint" "Custom_LED_THT:LED_D5.0mm" (at 90.17 83.82 0)
       (effects (font (size 1.27 1.27)) hide)
     )
@@
       (effects (font (size 1.27 1.27)) (justify left))
     )
-    (property "Footprint" "TestPoint:TestPoint_Pad_D1.5mm" (at 144.78 78.74 0)
+    (property "Footprint" "Xaar-Driver:TestPoint_Pad_D1.5mm" (at 144.78 78.74 0)
       (effects (font (size 1.27 1.27)) hide)
     )
@@
       (effects (font (size 1.27 1.27)) (justify right))
     )
-    (property "Footprint" "LED_THT:LED_D5.0mm" (at 90.17 142.24 0)
+    (property "Footprint" "Custom_LED_THT:LED_D5.0mm" (at 90.17 142.24 0)
       (effects (font (size 1.27 1.27)) hide)
     )
@@
       (effects (font (size 1.27 1.27)) (justify right))
     )
-    (property "Footprint" "TestPoint:TestPoint_Pad_D1.5mm" (at 66.04 99.06 0)
+    (property "Footprint" "Xaar-Driver:TestPoint_Pad_D1.5mm" (at 66.04 99.06 0)
       (effects (font (size 1.27 1.27)) hide)
     )
@@
       (effects (font (size 1.27 1.27)) (justify right))
     )
-    (property "Footprint" "TestPoint:TestPoint_Pad_D1.5mm" (at 67.31 157.48 0)
-      (effects (font (size 1.27 1.27)) hide)
-    )
+    (property "Footprint" "Xaar-Driver:TestPoint_Pad_D1.5mm" (at 67.31 157.48 0)
+      (effects (font (size 1.27 1.27)) hide)
+    )

Commit message: add acc and text
Parts:
- C7: value (none) -> 100n >16V Cer
Changed lines of the file:
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@@
       (effects (font (size 1.27 1.27)))
     )
-    (property "Value" "  " (at 220.98 21.59 90)
+    (property "Value" "100n >16V Cer" (at 220.98 21.59 90)
       (effects (font (size 1.27 1.27)))
     )

Commit message: create order list
Parts:
- R6: footprint Resistor_SMD:R_0603_1608Metric_Pad0.98x0.95mm_HandSolder -> Resistor_SMD:R_0805_2012Metric_Pad1.20x1.40mm_HandSolder; RSBestNr 198-5552 -> 721-7804
Changed lines of the file:
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@@
       (effects (font (size 1.27 1.27)) (justify left))
     )
-    (property "Footprint" "Resistor_SMD:R_0603_1608Metric_Pad0.98x0.95mm_HandSolder" (at 35.052 73.66 90)
+    (property "Footprint" "Resistor_SMD:R_0805_2012Metric_Pad1.20x1.40mm_HandSolder" (at 35.052 73.66 90)
       (effects (font (size 1.27 1.27)) hide)
     )
@@
       (effects (font (size 1.27 1.27)) hide)
     )
-    (property "RSBestNr" "198-5552" (at 36.83 73.66 0)
+    (property "RSBestNr" "721-7804" (at 36.83 73.66 0)
       (effects (font (size 1.27 1.27)) hide)
     )

Commit message: fix dac address r
Parts:
- renumbered D4 to D3, D5 to D4, NT3 to NT4, Q3 to Q10, Q7 to Q11, R11 to R10, R14 to R11, R3 to R12, R12 to R13, R16 to R14, R17 to R15, R13 to R16, R15 to R17, R4 to R2, R3 to R22, R6 to R3, R7 to R4, R17 to R45, R14 to R46, R17 to R49, R2 to R5, R9 to R6, R5 to R7, R10 to R8, R8 to R9

Commit message: fix nmos
Parts:
- Q1, Q2: value DMN2075U -> DMN5L06K-7
Changed lines of the file:
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@@
 			)
 		)
-		(property "Value" "DMN2075U"
+		(property "Value" "DMN5L06K-7"
 			(at 93.98 100.33 0)
 			(effects
@@
 			)
 		)
-		(property "Value" "DMN2075U"
+		(property "Value" "DMN5L06K-7"
 			(at 93.98 158.75 0)
 			(effects
