File: Xaar128-Driver/Xaar128-Driver.kicad_pcb (KiCad board)
At the start: 2 copper layers, 100 x 100 mm, 169 parts, among them J1 Screw_Terminal_01x02, J3 Screw_Terminal_01x02, J4 Screw_Terminal_01x02, J5 Conn_01x21, J7 Screw_Terminal_01x04, Q1 DMN2075U, Q10 DMN2075U, Q11 DMG2305UX, Q2 DMN2075U, Q3 DMN2075U, Q4 DMN2075U, Q5 DMN2075U, Q6 DMN2075U, Q7 DMG2305UX, Q8 DMG2305UX, Q9 DMN2075U, U1 6N135, U10 74AHCT125, U11 LM317_TO-220, U12 TXB0104D, U13 MCP4725xxx-xCH, U14 ISO1540, U15 L7824, U16 MC78L05_SOT89, U17 TLC272, U18 MCP3021, U19 LTV-356T, U2 6N135, U20 74AHCT125, U21 74HC173, U3 74HC173, U4 NUCLEO-H743ZI2, U5 TXB0104D, U6 TXB0104D, U7 TXB0104D, U8 74AHCT125, U9 74AHCT125

Commit message: routing done
Parts:
- C17, C19: value 1u >72V E -> 2.2u >72V E; footprint Capacitor_THT:CP_Radial_D8.0mm_P3.50mm -> Capacitor_THT:CP_Radial_D5.0mm_P2.00mm
- NT3: moved to F.Cu
- moved R31 68.7 mm to (105.7, 86.9), turned to 90 degrees
- moved R32 68.6 mm to (104.6, 90.9), turned to 180 degrees
- moved TP6 58.9 mm to (119.9, 112.3)
- moved R39 57.6 mm to (106.9, 102.6)
- moved R37 54.8 mm to (112.3, 97.8)
- moved TP7 53.2 mm to (111.0, 102.1)
- moved JP2 52.8 mm to (114.8, 95.3), turned to 0 degrees
- moved NT1 52.4 mm to (122.9, 104.4)
- moved R38 52.2 mm to (112.3, 101.1), turned to 90 degrees
- moved R40 51.1 mm to (97.8, 97.3)
- moved TP8 49.0 mm to (110.0, 97.5)
- moved C18 46.1 mm to (114.0, 91.6)
- moved R30 44.1 mm to (118.4, 99.6)
- moved D10 38.6 mm to (121.7, 102.4)
- moved NT7 22.4 mm to (51.3, 85.9)
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Connections:
- U12 pad 12: /Level Shift/RESET_DISABLE_CP_OUT -> /HV Supply/VPP_ENABLE_CP_5
- U12 pad 13: /HV Supply/VPP_ENABLE_CP_5 -> /Level Shift/RESET_DISABLE_CP_OUT
- U12 pad 2: /Level Shift/VPP_EN_CP_IN -> /Level Shift/RESET_DISABLE_CP_IN
- U12 pad 3: /Level Shift/RESET_DISABLE_CP_IN -> /Level Shift/VPP_EN_CP_IN
- U20 pad 11: /Level Shift/RESET_DISABLE_CP_OUT -> /HV Supply/VPP_ENABLE_CP_5
- U20 pad 12: /Level Shift/RESET_DISABLE_CP_IN -> /Level Shift/VPP_EN_CP_IN
- U20 pad 2: /Level Shift/VPP_EN_CP_IN -> /Level Shift/RESET_DISABLE_CP_IN
- U20 pad 3: /HV Supply/VPP_ENABLE_CP_5 -> /Level Shift/RESET_DISABLE_CP_OUT
Routing:
- net GND1: track 260.0 -> 311.1 mm, vias 7 -> 11
- net GND: track 508.9 -> 546.2 mm
- net Net-(U13-VOUT): track 7.01 -> 44.2 mm, vias 0 -> 1
- net +5V: track 241.0 -> 273.8 mm, vias 7 -> 9
- net +5VP: track 68.4 -> 85.7 mm, vias 0 -> 2
- net Net-(D10-A): track 12.7 -> 28.2 mm
- net Net-(JP2-A): track 19.5 -> 8.90 mm
- net Net-(R38-Pad1): track 18.3 -> 11.5 mm
- net Net-(R31-Pad1): track 2.35 -> 8.88 mm
- net /IO/LED-: track 18.9 -> 24.4 mm, vias 0 -> 2
- net /Level Shift/RESET_DISABLE_CP_IN: track 34.1 -> 38.9 mm, vias 2 -> 3
- net Net-(Q2-G): track 3.31 -> 7.02 mm, vias 0 -> 1
- net Net-(Q1-G): track 2.13 -> 5.71 mm, vias 0 -> 1
- net Net-(U21-Q0): track 2.12 -> 5.49 mm, vias 0 -> 1
- net Net-(U18-AIN): track 6.19 -> 9.21 mm, vias 0 -> 1
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