File: Xaar128-Driver/Xaar128-Driver.kicad_pcb (KiCad board)
At the start: 2 copper layers, 100 x 100 mm, 169 parts, among them J1 Screw_Terminal_01x02, J3 Screw_Terminal_01x02, J4 Screw_Terminal_01x02, J5 Conn_01x21, J7 Screw_Terminal_01x04, Q1 DMN2075U, Q10 DMN2075U, Q11 DMG2305UX, Q2 DMN2075U, Q3 DMN2075U, Q4 DMN2075U, Q5 DMN2075U, Q6 DMN2075U, Q7 DMG2305UX, Q8 DMG2305UX, Q9 DMN2075U, U1 6N135, U10 74AHCT125, U11 LM317_TO-220, U12 TXB0104D, U13 MCP4725xxx-xCH, U14 ISO1540, U15 L7824, U16 MC78L05_SOT89, U17 TLC272, U18 MCP3021, U19 LTV-356T, U2 6N135, U20 74AHCT125, U21 74HC173, U3 74HC173, U4 NUCLEO-H743ZI2, U5 TXB0104D, U6 TXB0104D, U7 TXB0104D, U8 74AHCT125, U9 74AHCT125

Commit message: drc & plots done
Parts:
- added H1: MountingHole, MountingHole:MountingHole_2.7mm_M2.5_DIN965, F.Cu at (36.0, 176.8)
- added H2: MountingHole, MountingHole:MountingHole_2.7mm_M2.5_DIN965, F.Cu at (92.0, 86.8)
- added H3: MountingHole, MountingHole:MountingHole_2.7mm_M2.5_DIN965, F.Cu at (127.0, 132.8)
- added H4: MountingHole, MountingHole:MountingHole_2.7mm_M2.5_DIN965, F.Cu at (37.8, 152.5)
- added J2: Screw_Terminal_01x02, RS_PRO:897-1051, F.Cu at (59.9, 89.7)
- D3, D4: footprint LED_THT:LED_D5.0mm -> Custom_LED_THT:LED_D5.0mm
- J1, J3, J4: footprint RS_PRO:Steckbarer_Klemmenblock_1x02_5.08mm_vertical -> RS_PRO:897-1051
- J7: value Screw_Terminal_01x04 -> Screw_Terminal_01x02; footprint RS_PRO:Steckbarer_Klemmenblock_1x04_5.08mm_vertical_copy -> RS_PRO:897-1051
- TP1, TP10, TP11, TP12, TP13, TP2, TP3, TP4, TP5, TP6, TP7, TP8, TP9: footprint TestPoint:TestPoint_Pad_D1.5mm -> Xaar-Driver:TestPoint_Pad_D1.5mm
- U16: footprint Package_TO_SOT_SMD:SOT-89-3 -> Xaar-Driver:SOT-89-3
- moved JP13 10.5 mm to (44.6, 123.4), turned to 180 degrees
- moved J7 3.94 mm to (49.8, 89.7)
- moved J4 3.82 mm to (70.1, 89.7)
- moved J3 3.56 mm to (121.7, 89.3)
- moved NT7 2.05 mm to (51.6, 87.9)
- moved NT4 1.78 mm to (130.0, 99.8)
- moved HS1 1.62 mm to (153.9, 96.0)
- moved U11 1.62 mm to (127.3, 93.7)
- moved NT3 1.03 mm to (125.0, 98.6)
- moved TP11 0.68 mm to (121.2, 153.9)
- moved J1 0.49 mm to (39.0, 164.6)
Routing:
- net GND: track 546.2 -> 524.9 mm
- net /Level Shift/CLK_IN: track 73.4 -> 52.3 mm
- net GND1: track 311.1 -> 298.1 mm
- net Net-(JP13-B): track 3.15 -> 13.2 mm
- net +5V: track 273.8 -> 269.5 mm
- net /IO/LED-: track 24.4 -> 21.1 mm
- net +36V: track 32.3 -> 35.3 mm
- net /MCU/SDA: track 127.8 -> 125.0 mm
- net /MCU/SCL: track 136.7 -> 134.1 mm
- net SDA_HV: track 61.3 -> 63.7 mm
- net Net-(D7-A): track 54.6 -> 56.5 mm
- net Net-(D10-A): track 28.2 -> 29.9 mm
- net Net-(NT4-Pad2): track 45.4 -> 43.9 mm
- net /HV Supply/VPP: track 18.6 -> 20.1 mm
- net Net-(U15-IN): track 11.7 -> 12.7 mm
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
Commit message: add acc and text
Parts:
- added C33: 100n >16V Cer, Capacitor_SMD:C_0603_1608Metric_Pad1.08x0.95mm_HandSolder, B.Cu at (80.3, 104.8)
- added JP17: SolderJumper_2_Open, Resistor_SMD:R_0603_1608Metric_Pad0.98x0.95mm_HandSolder, B.Cu at (99.1, 112.3)
- added JP18: SolderJumper_2_Open, Resistor_SMD:R_0603_1608Metric_Pad0.98x0.95mm_HandSolder, B.Cu at (66.0, 108.2)
- added JP19: SolderJumper_2_Open, Resistor_SMD:R_0603_1608Metric_Pad0.98x0.95mm_HandSolder, B.Cu at (70.1, 104.1)
- added JP20: SolderJumper_2_Open, Resistor_SMD:R_0603_1608Metric_Pad0.98x0.95mm_HandSolder, B.Cu at (68.6, 106.2)
- added NT2: NetTie_2, NetTie:NetTie-2_SMD_Pad0.5mm, B.Cu at (71.1, 109.0)
- added NT5: NetTie_2, NetTie:NetTie-2_SMD_Pad0.5mm, B.Cu at (76.2, 110.5)
- added R47: 10k, Resistor_SMD:R_0603_1608Metric_Pad0.98x0.95mm_HandSolder, B.Cu at (78.7, 104.8)
- added R48: 10k, Resistor_SMD:R_0603_1608Metric_Pad0.98x0.95mm_HandSolder, B.Cu at (72.7, 103.9)
- added R53: 10k, Resistor_SMD:R_0603_1608Metric_Pad0.98x0.95mm_HandSolder, B.Cu at (76.2, 103.9)
- added TP14: TestPoint, Xaar-Driver:TestPoint_Pad_D1.5mm, F.Cu at (79.8, 111.5)
- added TP15: TestPoint, Xaar-Driver:TestPoint_Pad_D1.5mm, F.Cu at (79.8, 108.7)
- added U22: LIS2DH, Package_LGA:LGA-14_2x2mm_P0.35mm_LayoutBorder3x4y, B.Cu at (73.8, 109.9)
- C1, C10, C2, C21, C22, C23, C24, C26, C28, C29, C3, C30, C31, C4, C5, C6, C7, C8, C9: value (none) -> 100n >16V Cer
Connections:
- net /MCU/SCL renamed /ACC/SCL
- net /MCU/SDA renamed /ACC/SDA
Routing:
- net Net-(JP17-A): track 0.00 -> 44.4 mm, vias 0 -> 2
- net Net-(JP18-B): track 0.00 -> 24.8 mm, vias 0 -> 4
- net Net-(NT2-Pad1): track 0.00 -> 15.4 mm
- net +3.3V: track 132.8 -> 146.1 mm, vias 6 -> 8
- net Net-(U22-SDO): track 0.00 -> 7.43 mm
- net +5V: track 269.5 -> 275.8 mm
- net Net-(U22-INT1): track 0.00 -> 6.19 mm, vias 0 -> 1
- net Net-(U22-INT2): track 0.00 -> 6.15 mm, vias 0 -> 1
- net /ACC/SCL: track 134.1 -> 140.0 mm, vias 2 -> 4
- net Net-(JP19-A): track 0.00 -> 5.88 mm
- net Net-(U22-~{CS}): track 0.00 -> 5.82 mm
- net Net-(JP20-A): track 0.00 -> 5.59 mm
- net Net-(U22-Vdd): track 0.00 -> 3.21 mm
- net /ACC/SDA: track 125.0 -> 125.8 mm
- net GND1: track 298.1 -> 298.8 mm
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Other:
- board text added: "36V"
- board text added: "36V:MON:EN"
- board text added: "36V:MON:G"
- board text added: "5V"
- board text added: "5V:MON"
- board text added: "5V_MON_EN"
- board text added: "ADC"
- board text added: "ADJ"
- board text added: "AMP"
- board text added: "COMM_ENABLE"
- board text added: "DAC"
- board text added: "GND"
- board text added: "GND1"
- board text added: "LED+"
- board text added: "LED-"
- board text added: "LED_PWR"
- board text added: "LED_PWR_GND"
- board text added: "MCU"
- board text added: "POT"
- board text added: "Printhead Driver V1"
- board text added: "RESET:MON:EN"
- board text added: "SCL"
- board text added: "SDA"
- board text added: "VPP"
- board text added: "VPP:MON:EN"
- board text added: "VPP:MON:G"
- board text added: "VPP:OPTO:C"
- board text added: "VPP_EN:G"
- board text added: "nFAULT:MON:EN"
- board text added: "nFIRE"
- board text added: "nRESET"
- board text added: "nRESET_FAULT"

Commit message: create order list
Parts:
- R28, R3: footprint Resistor_SMD:R_0603_1608Metric_Pad0.98x0.95mm_HandSolder -> Resistor_SMD:R_0805_2012Metric_Pad1.20x1.40mm_HandSolder

Commit message: Create plots for fabrication
Changed lines of the file:
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@@
     (property "ki_keywords" "R res resistor")
     (attr smd)
-    (fp_text reference "R28" (at 0 1.65 270) (layer "B.SilkS")
+    (fp_text reference "R28" (at 3.3865 -0.004 270) (layer "B.SilkS")
         (effects (font (size 1 1) (thickness 0.15)) (justify mirror))
     )
@@
     (fp_line (start 1 0.625) (end 1 -0.625)
       (stroke (width 0.1) (type solid)) (layer "B.Fab"))
-    (pad "1" smd roundrect (at -1 0 90) (size 1.2 1.4) (layers "B.Cu" "B.Paste" "B.Mask") (roundrect_rratio 0.208333)
+    (pad "1" smd roundrect (at -1 0 90) (size 1.2 1.4) (layers "B.Cu" "B.Paste" "B.Mask") (roundrect_rratio 0.2083333333)
       (net 3 "/HV Supply/VPP_Feedback") (pintype "passive"))
-    (pad "2" smd roundrect (at 1 0 90) (size 1.2 1.4) (layers "B.Cu" "B.Paste" "B.Mask") (roundrect_rratio 0.208333)
+    (pad "2" smd roundrect (at 1 0 90) (size 1.2 1.4) (layers "B.Cu" "B.Paste" "B.Mask") (roundrect_rratio 0.2083333333)
       (net 25 "Net-(D9-A)") (pintype "passive"))
     (model "${KICAD6_3DMODEL_DIR}/Resistor_SMD.3dshapes/R_0805_2012Metric.wrl"
@@
     (fp_line (start 1 0.625) (end 1 -0.625)
       (stroke (width 0.1) (type solid)) (layer "B.Fab"))
-    (pad "1" smd roundrect (at -1 0) (size 1.2 1.4) (layers "B.Cu" "B.Paste" "B.Mask") (roundrect_rratio 0.208333)
+    (pad "1" smd roundrect (at -1 0) (size 1.2 1.4) (layers "B.Cu" "B.Paste" "B.Mask") (roundrect_rratio 0.2083333333)
       (net 29 "/HV Supply/VPPL") (pintype "passive"))
-    (pad "2" smd roundrect (at 1 0) (size 1.2 1.4) (layers "B.Cu" "B.Paste" "B.Mask") (roundrect_rratio 0.208333)
+    (pad "2" smd roundrect (at 1 0) (size 1.2 1.4) (layers "B.Cu" "B.Paste" "B.Mask") (roundrect_rratio 0.2083333333)
       (net 15 "Net-(D1-K)") (pintype "passive"))
     (model "${KICAD6_3DMODEL_DIR}/Resistor_SMD.3dshapes/R_0805_2012Metric.wrl"

Commit message: ordering voltage regulator extension
Parts:
- U14: value ISO1540 -> ISO1541

Commit message: fix dac address r
Parts:
- added R60: 10k, Resistor_SMD:R_0603_1608Metric_Pad0.98x0.95mm_HandSolder, B.Cu at (126.0, 123.7)
Connections:
- U13 pad 6: unconnected-(U13-A0-Pad6) -> Net-(U13-A0)
Routing:
- net GND1: track 298.8 -> 319.9 mm
- net Net-(U13-A0): track 0.00 -> 2.33 mm
- net SCL_HV: track 67.9 -> 68.6 mm

Commit message: switch opv to lm358
Parts:
- U17: value TLC272 -> LM358
Changed lines of the file:
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@@
 		(fp_arc
 			(start 36.273976 109.758869)
-			(mid 35.688183 111.173077)
+			(mid 35.688183 111.173081)
 			(end 34.273973 111.75887)
 			(stroke
@@
 		(fp_arc
 			(start 34.273975 -21.58113)
-			(mid 35.68818 -20.995348)
+			(mid 35.688216 -20.995354)
 			(end 36.273976 -19.581129)
 			(stroke
@@
 		(fp_arc
 			(start -10.953202 110.157502)
-			(mid -10.528202 109.732505)
+			(mid -10.528202 109.732506)
 			(end -10.103201 110.157502)
 			(stroke
@@
 			)
 		)
-		(property "Value" "TLC272"
+		(property "Value" "LM358"
 			(at 3.81 9.95 90)
 			(layer "F.Fab")
@@
 		(tags "resistor handsolder")
 		(property "Reference" "R60"
-			(at 0 1.43 360)
+			(at 0 1.43 0)
 			(layer "B.SilkS")
 			(effects
@@
 		)
 		(property "Value" "10k"
-			(at 0 -1.43 360)
+			(at 0 -1.43 0)
 			(layer "B.Fab")
 			(effects
@@
 		)
 		(fp_text user "${REFERENCE}"
-			(at 0 0 360)
+			(at 0 0 0)
 			(layer "B.Fab")
 			(effects
