File: Xaar128-Driver/level_shift.kicad_sch (KiCad schematic)
At the start: 28 parts, among them Q1 DMN2075U, U10 74AHCT125, U12 TXB0104D, U20 74AHCT125, U5 TXB0104D, U6 TXB0104D, U7 TXB0104D, U8 74AHCT125, U9 74AHCT125

Commit message: more routing
Connections:
- net RESET_DISABLE_CP_IN: now also U12.3 (A2), U20.12 (4A); no longer U12.2 (A1), U20.2 (1A)
- net RESET_DISABLE_CP_OUT: now also U12.12 (B2), U20.11 (4Y); no longer U12.13 (B1), U20.3 (1Y)
- net VPP_EN_CP_IN: now also U12.2 (A1), U20.2 (1A); no longer U12.3 (A2), U20.12 (4A)
- net VPP_EN_CP_OUT: now also U12.13 (B1), U20.3 (1Y); no longer U12.12 (B2), U20.11 (4Y)
Changed lines of the file:
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@@
+    (effects (font (size 1.27 1.27)) (justify left))
+  )
+  (hierarchical_label "VPP_EN_CP_OUT" (shape output) (at 255.27 46.99 0) (fields_autoplaced)
     (effects (font (size 1.27 1.27)) (justify left))
   )
@@
     (effects (font (size 1.27 1.27)) (justify left))
   )
-  (hierarchical_label "RESET_DISABLE_CP_IN" (shape input) (at 234.95 46.99 180) (fields_autoplaced)
-    (effects (font (size 1.27 1.27)) (justify right))
-  )
   (hierarchical_label "READY_OUT" (shape output) (at 189.23 60.96 0) (fields_autoplaced)
     (effects (font (size 1.27 1.27)) (justify left))
@@
   )
   (hierarchical_label "nFIRE_IN" (shape input) (at 101.6 55.88 180) (fields_autoplaced)
+    (effects (font (size 1.27 1.27)) (justify right))
+  )
+  (hierarchical_label "VPP_EN_CP_IN" (shape input) (at 234.95 46.99 180) (fields_autoplaced)
+    (effects (font (size 1.27 1.27)) (justify right))
+  )
+  (hierarchical_label "RESET_DISABLE_CP_IN" (shape input) (at 232.41 106.68 180) (fields_autoplaced)
     (effects (font (size 1.27 1.27)) (justify right))
   )
@@
     (effects (font (size 1.27 1.27)) (justify left))
   )
-  (hierarchical_label "VPP_EN_CP_IN" (shape input) (at 232.41 106.68 180) (fields_autoplaced)
-    (effects (font (size 1.27 1.27)) (justify right))
-  )
   (hierarchical_label "MOSI_IN" (shape input) (at 36.83 59.69 180) (fields_autoplaced)
-    (effects (font (size 1.27 1.27)) (justify right))
-  )
-  (hierarchical_label "VPP_EN_CP_IN" (shape input) (at 234.95 52.07 180) (fields_autoplaced)
     (effects (font (size 1.27 1.27)) (justify right))
   )
@@
     (effects (font (size 1.27 1.27)) (justify left))
   )
+  (hierarchical_label "VPP_EN_CP_OUT" (shape output) (at 257.81 99.06 0) (fields_autoplaced)
+    (effects (font (size 1.27 1.27)) (justify left))
+  )
   (hierarchical_label "nFIRE_OUT" (shape output) (at 123.19 100.33 0) (fields_autoplaced)
     (effects (font (size 1.27 1.27)) (justify left))
@@
     (effects (font (size 1.27 1.27)) (justify right))
   )
+  (hierarchical_label "RESET_DISABLE_CP_OUT" (shape output) (at 255.27 52.07 0) (fields_autoplaced)
+    (effects (font (size 1.27 1.27)) (justify left))
+  )
   (hierarchical_label "PHO_IN" (shape input) (at 34.29 97.79 180) (fields_autoplaced)
     (effects (font (size 1.27 1.27)) (justify right))
@@
     (effects (font (size 1.27 1.27)) (justify right))
   )
-  (hierarchical_label "RESET_DISABLE_CP_OUT" (shape output) (at 257.81 99.06 0) (fields_autoplaced)
-    (effects (font (size 1.27 1.27)) (justify left))
-  )
   (hierarchical_label "nFIRE_OUT" (shape output) (at 121.92 55.88 0) (fields_autoplaced)
     (effects (font (size 1.27 1.27)) (justify left))
@@
   (hierarchical_label "CLK_OUT" (shape output) (at 121.92 50.8 0) (fields_autoplaced)
     (effects (font (size 1.27 1.27)) (justify left))
+  )
+  (hierarchical_label "RESET_DISABLE_CP_IN" (shape input) (at 234.95 52.07 180) (fields_autoplaced)
+    (effects (font (size 1.27 1.27)) (justify right))
   )
   (hierarchical_label "SCK_OUT" (shape output) (at 57.15 54.61 0) (fields_autoplaced)
@@
     (effects (font (size 1.27 1.27)) (justify right))
   )
+  (hierarchical_label "RESET_DISABLE_CP_OUT" (shape output) (at 257.81 106.68 0) (fields_autoplaced)
+    (effects (font (size 1.27 1.27)) (justify left))
+  )
   (hierarchical_label "nSS2_OUT" (shape output) (at 123.19 97.79 0) (fields_autoplaced)
     (effects (font (size 1.27 1.27)) (justify left))
@@
     (effects (font (size 1.27 1.27)) (justify right))
   )
-  (hierarchical_label "VPP_EN_CP_OUT" (shape output) (at 257.81 106.68 0) (fields_autoplaced)
-    (effects (font (size 1.27 1.27)) (justify left))
-  )
   (hierarchical_label "nSS2_OUT" (shape output) (at 121.92 45.72 0) (fields_autoplaced)
     (effects (font (size 1.27 1.27)) (justify left))
   )
   (hierarchical_label "nRESET_FAULT_IN" (shape input) (at 166.37 97.79 180) (fields_autoplaced)
-    (effects (font (size 1.27 1.27)) (justify right))
-  )
-  (hierarchical_label "RESET_DISABLE_CP_IN" (shape input) (at 232.41 99.06 180) (fields_autoplaced)
     (effects (font (size 1.27 1.27)) (justify right))
   )
@@
     (effects (font (size 1.27 1.27)) (justify right))
   )
-  (hierarchical_label "RESET_DISABLE_CP_OUT" (shape output) (at 255.27 46.99 0) (fields_autoplaced)
-    (effects (font (size 1.27 1.27)) (justify left))
+  (hierarchical_label "VPP_EN_CP_IN" (shape input) (at 232.41 99.06 180) (fields_autoplaced)
+    (effects (font (size 1.27 1.27)) (justify right))
   )
   (hierarchical_label "nFAULT_IN" (shape input) (at 168.91 50.8 180) (fields_autoplaced)
     (effects (font (size 1.27 1.27)) (justify right))
   )
-  (hierarchical_label "VPP_EN_CP_OUT" (shape output) (at 255.27 52.07 0) (fields_autoplaced)
-    (effects (font (size 1.27 1.27)) (justify left))
-  )
   (hierarchical_label "nSS1_IN" (shape input) (at 36.83 49.53 180) (fields_autoplaced)

Commit message: routing done
Connections:
- net RESET_DISABLE_CP_IN: now also U12.2 (A1), U20.2 (1A); no longer U12.3 (A2), U20.12 (4A)
- net RESET_DISABLE_CP_OUT: now also U12.13 (B1), U20.3 (1Y); no longer U12.12 (B2), U20.11 (4Y)
- net VPP_EN_CP_IN: now also U12.3 (A2), U20.12 (4A); no longer U12.2 (A1), U20.2 (1A)
- net VPP_EN_CP_OUT: now also U12.12 (B2), U20.11 (4Y); no longer U12.13 (B1), U20.3 (1Y)
Changed lines of the file:
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@@
+    (effects (font (size 1.27 1.27)) (justify right))
+  )
+  (hierarchical_label "RESET_DISABLE_CP_IN" (shape input) (at 232.41 99.06 180) (fields_autoplaced)
     (effects (font (size 1.27 1.27)) (justify right))
   )
@@
     (effects (font (size 1.27 1.27)) (justify left))
   )
-  (hierarchical_label "VPP_EN_CP_OUT" (shape output) (at 255.27 46.99 0) (fields_autoplaced)
+  (hierarchical_label "nRESET_IN" (shape input) (at 104.14 154.94 0) (fields_autoplaced)
     (effects (font (size 1.27 1.27)) (justify left))
   )
-  (hierarchical_label "nRESET_IN" (shape input) (at 104.14 154.94 0) (fields_autoplaced)
+  (hierarchical_label "VPP_EN_CP_OUT" (shape output) (at 257.81 106.68 0) (fields_autoplaced)
     (effects (font (size 1.27 1.27)) (justify left))
   )
@@
   )
   (hierarchical_label "nFIRE_IN" (shape input) (at 101.6 55.88 180) (fields_autoplaced)
-    (effects (font (size 1.27 1.27)) (justify right))
-  )
-  (hierarchical_label "VPP_EN_CP_IN" (shape input) (at 234.95 46.99 180) (fields_autoplaced)
-    (effects (font (size 1.27 1.27)) (justify right))
-  )
-  (hierarchical_label "RESET_DISABLE_CP_IN" (shape input) (at 232.41 106.68 180) (fields_autoplaced)
     (effects (font (size 1.27 1.27)) (justify right))
   )
@@
     (effects (font (size 1.27 1.27)) (justify left))
   )
-  (hierarchical_label "VPP_EN_CP_OUT" (shape output) (at 257.81 99.06 0) (fields_autoplaced)
-    (effects (font (size 1.27 1.27)) (justify left))
-  )
   (hierarchical_label "nFIRE_OUT" (shape output) (at 123.19 100.33 0) (fields_autoplaced)
     (effects (font (size 1.27 1.27)) (justify left))
@@
     (effects (font (size 1.27 1.27)) (justify right))
   )
-  (hierarchical_label "RESET_DISABLE_CP_OUT" (shape output) (at 255.27 52.07 0) (fields_autoplaced)
+  (hierarchical_label "RESET_DISABLE_CP_OUT" (shape output) (at 255.27 46.99 0) (fields_autoplaced)
     (effects (font (size 1.27 1.27)) (justify left))
   )
@@
     (effects (font (size 1.27 1.27)) (justify right))
   )
+  (hierarchical_label "RESET_DISABLE_CP_IN" (shape input) (at 234.95 46.99 180) (fields_autoplaced)
+    (effects (font (size 1.27 1.27)) (justify right))
+  )
   (hierarchical_label "nFIRE_OUT" (shape output) (at 121.92 55.88 0) (fields_autoplaced)
     (effects (font (size 1.27 1.27)) (justify left))
@@
   (hierarchical_label "CLK_OUT" (shape output) (at 121.92 50.8 0) (fields_autoplaced)
     (effects (font (size 1.27 1.27)) (justify left))
-  )
-  (hierarchical_label "RESET_DISABLE_CP_IN" (shape input) (at 234.95 52.07 180) (fields_autoplaced)
-    (effects (font (size 1.27 1.27)) (justify right))
   )
   (hierarchical_label "SCK_OUT" (shape output) (at 57.15 54.61 0) (fields_autoplaced)
@@
     (effects (font (size 1.27 1.27)) (justify left))
   )
+  (hierarchical_label "RESET_DISABLE_CP_OUT" (shape output) (at 257.81 99.06 0) (fields_autoplaced)
+    (effects (font (size 1.27 1.27)) (justify left))
+  )
   (hierarchical_label "nSS1_OUT" (shape output) (at 59.69 105.41 0) (fields_autoplaced)
     (effects (font (size 1.27 1.27)) (justify left))
@@
     (effects (font (size 1.27 1.27)) (justify right))
   )
-  (hierarchical_label "RESET_DISABLE_CP_OUT" (shape output) (at 257.81 106.68 0) (fields_autoplaced)
-    (effects (font (size 1.27 1.27)) (justify left))
-  )
   (hierarchical_label "nSS2_OUT" (shape output) (at 123.19 97.79 0) (fields_autoplaced)
     (effects (font (size 1.27 1.27)) (justify left))
@@
     (effects (font (size 1.27 1.27)) (justify right))
   )
+  (hierarchical_label "VPP_EN_CP_OUT" (shape output) (at 255.27 52.07 0) (fields_autoplaced)
+    (effects (font (size 1.27 1.27)) (justify left))
+  )
   (hierarchical_label "nSS2_OUT" (shape output) (at 121.92 45.72 0) (fields_autoplaced)
     (effects (font (size 1.27 1.27)) (justify left))
   )
   (hierarchical_label "nRESET_FAULT_IN" (shape input) (at 166.37 97.79 180) (fields_autoplaced)
+    (effects (font (size 1.27 1.27)) (justify right))
+  )
+  (hierarchical_label "VPP_EN_CP_IN" (shape input) (at 232.41 106.68 180) (fields_autoplaced)
     (effects (font (size 1.27 1.27)) (justify right))
   )
@@
     (effects (font (size 1.27 1.27)) (justify right))
   )
-  (hierarchical_label "VPP_EN_CP_IN" (shape input) (at 232.41 99.06 180) (fields_autoplaced)
+  (hierarchical_label "VPP_EN_CP_IN" (shape input) (at 234.95 52.07 180) (fields_autoplaced)
     (effects (font (size 1.27 1.27)) (justify right))
   )
