File: Xaar128-Driver/level_shift.kicad_sch (KiCad schematic)
At the start: 28 parts, among them Q1 DMN2075U, U10 74AHCT125, U12 TXB0104D, U20 74AHCT125, U5 TXB0104D, U6 TXB0104D, U7 TXB0104D, U8 74AHCT125, U9 74AHCT125

Commit message: add acc and text
Parts:
- C1, C10, C2, C28, C29, C3, C30, C4, C5, C6, C8, C9: value (none) -> 100n >16V Cer
Changed lines of the file:
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@@
       (effects (font (size 1.27 1.27)))
     )
-    (property "Value" "  " (at 251.46 82.55 90)
+    (property "Value" "100n >16V Cer" (at 251.46 82.55 90)
       (effects (font (size 1.27 1.27)))
     )
@@
       (effects (font (size 1.27 1.27)))
     )
-    (property "Value" "  " (at 53.34 25.4 90)
+    (property "Value" "100n >16V Cer" (at 53.34 25.4 90)
       (effects (font (size 1.27 1.27)))
     )
@@
       (effects (font (size 1.27 1.27)))
     )
-    (property "Value" "  " (at 251.46 29.21 90)
+    (property "Value" "100n >16V Cer" (at 251.46 29.21 90)
       (effects (font (size 1.27 1.27)))
     )
@@
       (effects (font (size 1.27 1.27)))
     )
-    (property "Value" "  " (at 114.3 81.28 90)
+    (property "Value" "100n >16V Cer" (at 114.3 81.28 90)
       (effects (font (size 1.27 1.27)))
     )
@@
       (effects (font (size 1.27 1.27)))
     )
-    (property "Value" "  " (at 172.72 27.94 90)
+    (property "Value" "100n >16V Cer" (at 172.72 27.94 90)
       (effects (font (size 1.27 1.27)))
     )
@@
       (effects (font (size 1.27 1.27)))
     )
-    (property "Value" "  " (at 238.76 29.21 90)
+    (property "Value" "100n >16V Cer" (at 238.76 29.21 90)
       (effects (font (size 1.27 1.27)))
     )
@@
       (effects (font (size 1.27 1.27)))
     )
-    (property "Value" "  " (at 185.42 27.94 90)
+    (property "Value" "100n >16V Cer" (at 185.42 27.94 90)
       (effects (font (size 1.27 1.27)))
     )
@@
       (effects (font (size 1.27 1.27)))
     )
-    (property "Value" "  " (at 40.64 25.4 90)
+    (property "Value" "100n >16V Cer" (at 40.64 25.4 90)
       (effects (font (size 1.27 1.27)))
     )
@@
       (effects (font (size 1.27 1.27)))
     )
-    (property "Value" "  " (at 185.42 81.28 90)
+    (property "Value" "100n >16V Cer" (at 185.42 81.28 90)
       (effects (font (size 1.27 1.27)))
     )
@@
       (effects (font (size 1.27 1.27)))
     )
-    (property "Value" "  " (at 118.11 26.67 90)
+    (property "Value" "100n >16V Cer" (at 118.11 26.67 90)
       (effects (font (size 1.27 1.27)))
     )
@@
       (effects (font (size 1.27 1.27)))
     )
-    (property "Value" "  " (at 50.8 81.28 90)
+    (property "Value" "100n >16V Cer" (at 50.8 81.28 90)
       (effects (font (size 1.27 1.27)))
     )
@@
       (effects (font (size 1.27 1.27)))
     )
-    (property "Value" "  " (at 105.41 26.67 90)
-      (effects (font (size 1.27 1.27)))
-    )
+    (property "Value" "100n >16V Cer" (at 105.41 26.67 90)
+      (effects (font (size 1.27 1.27)))
+    )

Commit message: fix dac address r
Parts:
- renumbered Q1 to Q6
