File: Xaar128-Driver/regulator.kicad_sch (KiCad schematic)
At the start: 42 parts, among them U11 LM317_TO-220, U13 MCP4725xxx-xCH, U14 ISO1540, U15 L7824, U16 MC78L05_SOT89, U17 TLC272, U18 MCP3021

Commit message: some component selections, fix wrong mcu
Parts:
- C17, C19: value 1u -> 1u >72V E
- C18: value 10u -> 10u >72V E
- C20, C25: value 10u -> 10u > 16V Tantal; now not fitted
- C21, C22, C23, C24, C26: value 0.1u -> 100n >16V Cer; footprint (none) -> Capacitor_SMD:C_0603_1608Metric_Pad1.08x0.95mm_HandSolder; Supplier (none) -> Elektroplatz; now not fitted
- JP2: footprint (none) -> Connector_PinHeader_2.54mm:PinHeader_1x03_P2.54mm_Vertical; Funktion (none) -> Enable MCU Regulator Control
- NT1, NT3, NT4: footprint (none) -> NetTie:NetTie-2_SMD_Pad0.5mm; Supplier (none) -> None
- R33, R34, R35, R36, R41, R42, U15: now not fitted
- TP11: value SDA -> TestPoint; footprint (none) -> TestPoint:TestPoint_Pad_D1.5mm; Funktion (none) -> SDA; Supplier (none) -> None
- TP12: value SCL -> TestPoint; footprint (none) -> TestPoint:TestPoint_Pad_D1.5mm; Funktion (none) -> SCL; Supplier (none) -> None
- TP6: value V_DAC -> TestPoint; footprint (none) -> TestPoint:TestPoint_Pad_D1.5mm; Funktion (none) -> V_DAC; Supplier (none) -> None
- TP7: value V_DAC_AMP -> TestPoint; footprint (none) -> TestPoint:TestPoint_Pad_D1.5mm; Funktion (none) -> V_DAC_AMP; Supplier (none) -> None
- TP8: value V_ADJ -> TestPoint; footprint (none) -> TestPoint:TestPoint_Pad_D1.5mm; Funktion (none) -> V_ADJ; Supplier (none) -> None
- TP9: value V_ADC -> TestPoint; footprint (none) -> TestPoint:TestPoint_Pad_D1.5mm; Funktion (none) -> V_ADC; Supplier (none) -> None
- U11: RSBestNr (none) -> 661-6121; Supplier (none) -> RS
- U13: footprint Package_TO_SOT_SMD:SOT-23-6 -> Package_TO_SOT_SMD:SOT-23-6_Handsoldering; RSBestNr (none) -> 669-6290; Supplier (none) -> RS; now not fitted
- U14: RSBestNr (none) -> 825-3079; Supplier (none) -> RS; now not fitted
- U16: RSBestNr (none) -> 714-0679; Supplier (none) -> RS; now not fitted
- U17: Supplier (none) -> Elekroplatz; now not fitted
- U18: footprint MCP3021:SOT-23 -> Package_TO_SOT_SMD:SOT-23-5_HandSoldering; RSBestNr (none) -> 738-6011; Supplier (none) -> RS; now not fitted

Commit message: assign footprints
Parts:
- C17, C19: footprint (none) -> Capacitor_THT:CP_Radial_D8.0mm_P3.50mm; RSBestNr (none) -> 228-7265; Supplier (none) -> RS
- C18: footprint (none) -> Capacitor_SMD:CP_Elec_6.3x7.7; RSBestNr (none) -> 715-1442; Supplier (none) -> RS
- C20, C25: footprint (none) -> Capacitor_Tantalum_SMD:CP_EIA-3528-21_Kemet-B_Pad1.50x2.35mm_HandSolder; RSBestNr (none) -> 136-0203; Supplier (none) -> RS
- D11: value 1N4002 -> 1N4007; footprint (none) -> Diode_THT:D_DO-41_SOD81_P10.16mm_Horizontal; Supplier (none) -> Elektroplatz
- JP2: Supplier (none) -> Elektroplatz
- R33, R41: footprint (none) -> Resistor_SMD:R_0603_1608Metric_Pad0.98x0.95mm_HandSolder; RSBestNr (none) -> 678-9673; Supplier (none) -> RS
- R33: value 2.2k -> 2.2k > 600mW
- R33, R34, R35, R36: footprint (none) -> Resistor_SMD:R_0603_1608Metric_Pad0.98x0.95mm_HandSolder; Supplier (none) -> Elektroplatz
- R33: value 10k -> 4.7k
- RV1: value 4.7k -> 10k RC103B; footprint (none) -> Potentiometer_THT:Potentiometer_Alps_RK09L_Single_Vertical; Supplier (none) -> Elektroplatz
- U15: footprint (none) -> Package_TO_SOT_THT:TO-220-3_Vertical; RSBestNr (none) -> 298-8564; Supplier (none) -> RS
Other:
- note added: "V_pp = 1.25 * ( 1 + (R32 + (R31 * RV1/(R31 + RV1)))/R30) Output from 15-34.75 with nonlinearity - for better linearity, switch 10k and 4k7 (4k7k poti expensive..) minimum load current is 6.5mA, plus the leds and optocouplers at reset circuit should be enough"
- note removed: "V_pp = 1.25 * ( 1 + (R32 + (R31 * RV1/(R31 + RV1)))/R30) Output from 15-34.75 with slight nonlinearity minimum load current is 6.5mA, plus the leds and optocouplers at reset circuit should be enough"

Commit message: select remaining components, nucleo footprint
Parts:
- C18: footprint Capacitor_SMD:CP_Elec_6.3x7.7 -> Capacitor_THT:CP_Radial_D5.0mm_P2.00mm; RSBestNr 715-1442 -> 228-7079
- C21, C22, C23, C24, C26: value 100n >16V Cer -> (none)
- R33, R42: footprint (none) -> Resistor_SMD:R_1206_3216Metric_Pad1.30x1.75mm_HandSolder; RSBestNr (none) -> 812-1795; Supplier (none) -> RS
- R33: footprint (none) -> Resistor_SMD:R_2512_6332Metric_Pad1.40x3.35mm_HandSolder; RSBestNr (none) -> 755-1287; Supplier (none) -> RS
- R33: footprint (none) -> Resistor_SMD:R_0603_1608Metric_Pad0.98x0.95mm_HandSolder; RSBestNr (none) -> 901-3581; Supplier (none) -> RS
- R33: footprint (none) -> Resistor_THT:R_Axial_DIN0207_L6.3mm_D2.5mm_P7.62mm_Horizontal; Supplier (none) -> Elektroplatz
- R33: footprint (none) -> Resistor_THT:R_Axial_DIN0207_L6.3mm_D2.5mm_P7.62mm_Horizontal; RSBestNr (none) -> 148-332; Supplier (none) -> RS
Changed lines of the file:
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@@
       (effects (font (size 1.27 1.27)) (justify left))
     )
-    (property "Footprint" "Capacitor_SMD:CP_Elec_6.3x7.7" (at 216.8652 68.58 0)
+    (property "Footprint" "Capacitor_THT:CP_Radial_D5.0mm_P2.00mm" (at 216.8652 68.58 0)
       (effects (font (size 1.27 1.27)) hide)
     )
@@
       (effects (font (size 1.27 1.27)) hide)
     )
-    (property "RSBestNr" "715-1442" (at 215.9 64.77 0)
+    (property "RSBestNr" "228-7079" (at 215.9 64.77 0)
       (effects (font (size 1.27 1.27)) hide)
     )
@@
       (effects (font (size 1.27 1.27)) (justify left))
     )
-    (property "Footprint" "" (at 130.81 72.898 90)
+    (property "Footprint" "Resistor_SMD:R_1206_3216Metric_Pad1.30x1.75mm_HandSolder" (at 130.81 72.898 90)
       (effects (font (size 1.27 1.27)) hide)
     )
@@
       (effects (font (size 1.27 1.27)) hide)
     )
-    (property "RSBestNr" "" (at 130.81 71.12 0)
-      (effects (font (size 1.27 1.27)) hide)
-    )
-    (property "Supplier" "" (at 130.81 71.12 0)
+    (property "RSBestNr" "812-1795" (at 130.81 71.12 0)
+      (effects (font (size 1.27 1.27)) hide)
+    )
+    (property "Supplier" "RS" (at 130.81 71.12 0)
       (effects (font (size 1.27 1.27)) hide)
     )
@@
       (effects (font (size 1.27 1.27)))
     )
-    (property "Value" "100n >16V Cer" (at 66.04 130.81 90)
+    (property "Value" "  " (at 66.04 130.81 90)
       (effects (font (size 1.27 1.27)))
     )
@@
       (effects (font (size 1.27 1.27)) (justify left))
     )
-    (property "Footprint" "" (at 203.708 71.12 90)
+    (property "Footprint" "Resistor_SMD:R_2512_6332Metric_Pad1.40x3.35mm_HandSolder" (at 203.708 71.12 90)
       (effects (font (size 1.27 1.27)) hide)
     )
@@
       (effects (font (size 1.27 1.27)) hide)
     )
-    (property "RSBestNr" "" (at 201.93 71.12 0)
-      (effects (font (size 1.27 1.27)) hide)
-    )
-    (property "Supplier" "" (at 201.93 71.12 0)
+    (property "RSBestNr" "755-1287" (at 201.93 71.12 0)
+      (effects (font (size 1.27 1.27)) hide)
+    )
+    (property "Supplier" "RS" (at 201.93 71.12 0)
       (effects (font (size 1.27 1.27)) hide)
     )
@@
       (effects (font (size 1.27 1.27)))
     )
-    (property "Value" "100n >16V Cer" (at 78.74 64.77 90)
+    (property "Value" "  " (at 78.74 64.77 90)
       (effects (font (size 1.27 1.27)))
     )
@@
       (effects (font (size 1.27 1.27)) (justify left))
     )
-    (property "Footprint" "" (at 195.072 85.09 90)
+    (property "Footprint" "Resistor_SMD:R_0603_1608Metric_Pad0.98x0.95mm_HandSolder" (at 195.072 85.09 90)
       (effects (font (size 1.27 1.27)) hide)
     )
@@
       (effects (font (size 1.27 1.27)) hide)
     )
-    (property "RSBestNr" "" (at 196.85 85.09 0)
-      (effects (font (size 1.27 1.27)) hide)
-    )
-    (property "Supplier" "" (at 196.85 85.09 0)
+    (property "RSBestNr" "901-3581" (at 196.85 85.09 0)
+      (effects (font (size 1.27 1.27)) hide)
+    )
+    (property "Supplier" "RS" (at 196.85 85.09 0)
       (effects (font (size 1.27 1.27)) hide)
     )
@@
       (effects (font (size 1.27 1.27)) (justify left))
     )
-    (property "Footprint" "" (at 109.22 79.248 90)
+    (property "Footprint" "Resistor_THT:R_Axial_DIN0207_L6.3mm_D2.5mm_P7.62mm_Horizontal" (at 109.22 79.248 90)
       (effects (font (size 1.27 1.27)) hide)
     )
@@
       (effects (font (size 1.27 1.27)) hide)
     )
-    (property "Supplier" "" (at 109.22 77.47 0)
+    (property "Supplier" "Elektroplatz" (at 109.22 77.47 0)
       (effects (font (size 1.27 1.27)) hide)
     )
@@
       (effects (font (size 1.27 1.27)))
     )
-    (property "Value" "100n >16V Cer" (at 175.26 121.92 90)
+    (property "Value" "  " (at 175.26 121.92 90)
       (effects (font (size 1.27 1.27)))
     )
@@
       (effects (font (size 1.27 1.27)) (justify left))
     )
-    (property "Footprint" "" (at 214.122 43.18 90)
+    (property "Footprint" "Resistor_THT:R_Axial_DIN0207_L6.3mm_D2.5mm_P7.62mm_Horizontal" (at 214.122 43.18 90)
       (effects (font (size 1.27 1.27)) hide)
     )
@@
       (effects (font (size 1.27 1.27)) hide)
     )
-    (property "RSBestNr" "" (at 215.9 43.18 0)
-      (effects (font (size 1.27 1.27)) hide)
-    )
-    (property "Supplier" "" (at 215.9 43.18 0)
+    (property "RSBestNr" "148-332" (at 215.9 43.18 0)
+      (effects (font (size 1.27 1.27)) hide)
+    )
+    (property "Supplier" "RS" (at 215.9 43.18 0)
       (effects (font (size 1.27 1.27)) hide)
     )
@@
       (effects (font (size 1.27 1.27)))
     )
-    (property "Value" "100n >16V Cer" (at 119.38 62.23 90)
+    (property "Value" "  " (at 119.38 62.23 90)
       (effects (font (size 1.27 1.27)))
     )
@@
       (effects (font (size 1.27 1.27)))
     )
-    (property "Value" "100n >16V Cer" (at 44.45 130.81 90)
+    (property "Value" "  " (at 44.45 130.81 90)
       (effects (font (size 1.27 1.27)))
     )
@@
       (effects (font (size 1.27 1.27)) (justify left))
     )
-    (property "Footprint" "" (at 132.842 154.94 90)
+    (property "Footprint" "Resistor_SMD:R_1206_3216Metric_Pad1.30x1.75mm_HandSolder" (at 132.842 154.94 90)
       (effects (font (size 1.27 1.27)) hide)
     )
@@
       (effects (font (size 1.27 1.27)) hide)
     )
-    (property "RSBestNr" "" (at 134.62 154.94 0)
-      (effects (font (size 1.27 1.27)) hide)
-    )
-    (property "Supplier" "" (at 134.62 154.94 0)
-      (effects (font (size 1.27 1.27)) hide)
-    )
+    (property "RSBestNr" "812-1795" (at 134.62 154.94 0)
+      (effects (font (size 1.27 1.27)) hide)
+    )
+    (property "Supplier" "RS" (at 134.62 154.94 0)
+      (effects (font (size 1.27 1.27)) hide)
+    )

Commit message: xaar driver: some routed islands
Parts:
- removed NT4: NetTie_2, NetTie:NetTie-2_SMD_Pad0.5mm, symbol Device:NetTie_2
- added HS1: Heatsink, Xaar-Driver:SK68-375-SA, symbol Mechanical:Heatsink
Connections:
- net GND24 is gone; now on net GND1: R33.1, U15.2 (GND), U17.4 (V-)
- net +36V: now also NT3.2; no longer U15.1 (IN)
- net +5VP: now also U18.1 (VDD); no longer U18.P$1 (VCC)
- net GND1: now also C17.2, C19.2, C20.2, C21.2, C23.1, C25.2, C26.2, R42.2, U13.2 (VSS), U14.5 (GND2), U16.2 (GND), U18.2 (VSS)
- net SCL_HV: now also U18.5 (SCL); no longer U18.P$5 (SCL)
- net SDA_HV: now also U18.4 (SDA); no longer U18.P$4 (SDA)
- net at R41.2, R42.1, TP9.1: now also U18.3 (AIN); no longer U18.P$3 (AIN)
- removed net GND5HV: C20.2, C21.2, C23.1, C25.2, C26.2, NT3.1, R42.2, U13.2 (VSS), U14.5 (GND2), U16.2 (GND), U18.P$2 (GND)
- removed net GNDHP: C17.2, C19.2, NT3.2
- new net: NT3.1, U15.1 (IN)

Commit message: more routing
Changed lines of the file:
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@@
   (junction (at 124.46 33.02) (diameter 0) (color 0 0 0 0)
+  )
+  (junction (at 158.75 33.02) (diameter 0) (color 0 0 0 0)
   )
   (no_connect (at 52.07 85.09))
@@
     (stroke (width 0) (type default))
   )
-  (wire (pts (xy 157.48 33.02) (xy 161.29 33.02))
+  (wire (pts (xy 157.48 33.02) (xy 158.75 33.02))
     (stroke (width 0) (type default))
   )
@@
   )
   (wire (pts (xy 62.23 153.67) (xy 66.04 153.67))
+    (stroke (width 0) (type default))
+  )
+  (wire (pts (xy 158.75 33.02) (xy 161.29 33.02))
     (stroke (width 0) (type default))
   )
@@
         )
       )
+    )
+  )
+  (symbol (lib_id "power:PWR_FLAG") (at 158.75 33.02 180) (unit 1)
+    (in_bom yes) (on_board yes) (dnp no) (fields_autoplaced)
+    (property "Reference" "#FLG01" (at 158.75 34.925 0)
+      (effects (font (size 1.27 1.27)) hide)
+    )
+    (property "Value" "PWR_FLAG" (at 158.75 38.1 0)
+      (effects (font (size 1.27 1.27)))
+    )
+    (property "Footprint" "" (at 158.75 33.02 0)
+      (effects (font (size 1.27 1.27)) hide)
+    )
+    (property "Datasheet" "~" (at 158.75 33.02 0)
+      (effects (font (size 1.27 1.27)) hide)
+    )
+    (pin "1")
+    (instances
+      (project "Xaar128-Driver"
+        (path "/f0c82013-03f9-4093-aa02-30b89fd69529/48b639c9-d588-4ad3-b95b-9aa4a2d6905e"
+          (reference "#FLG01") (unit 1)
+        )
+      )

Commit message: routing done
Parts:
- C17, C19: value 1u >72V E -> 2.2u >72V E; footprint Capacitor_THT:CP_Radial_D8.0mm_P3.50mm -> Capacitor_THT:CP_Radial_D5.0mm_P2.00mm; RSBestNr 228-7265 -> 365-4442
Changed lines of the file:
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@@
       (effects (font (size 1.27 1.27)) (justify left))
     )
-    (property "Value" "1u >72V E" (at 250.19 49.911 0)
+    (property "Value" "2.2u >72V E" (at 250.19 49.911 0)
       (effects (font (size 1.27 1.27)) (justify left))
     )
-    (property "Footprint" "Capacitor_THT:CP_Radial_D8.0mm_P3.50mm" (at 247.3452 53.34 0)
+    (property "Footprint" "Capacitor_THT:CP_Radial_D5.0mm_P2.00mm" (at 247.3452 53.34 0)
       (effects (font (size 1.27 1.27)) hide)
     )
@@
       (effects (font (size 1.27 1.27)) hide)
     )
-    (property "RSBestNr" "228-7265" (at 246.38 49.53 0)
+    (property "RSBestNr" "365-4442" (at 246.38 49.53 0)
       (effects (font (size 1.27 1.27)) hide)
     )
@@
       (effects (font (size 1.27 1.27)) (justify left))
     )
-    (property "Value" "1u >72V E" (at 191.77 39.751 0)
+    (property "Value" "2.2u >72V E" (at 191.77 39.751 0)
       (effects (font (size 1.27 1.27)) (justify left))
     )
-    (property "Footprint" "Capacitor_THT:CP_Radial_D8.0mm_P3.50mm" (at 188.9252 43.18 0)
+    (property "Footprint" "Capacitor_THT:CP_Radial_D5.0mm_P2.00mm" (at 188.9252 43.18 0)
       (effects (font (size 1.27 1.27)) hide)
     )
@@
       (effects (font (size 1.27 1.27)) hide)
     )
-    (property "RSBestNr" "228-7265" (at 187.96 39.37 0)
+    (property "RSBestNr" "365-4442" (at 187.96 39.37 0)
       (effects (font (size 1.27 1.27)) hide)
     )

Commit message: drc & plots done
Parts:
- TP11, TP12, TP6, TP7, TP8, TP9: footprint TestPoint:TestPoint_Pad_D1.5mm -> Xaar-Driver:TestPoint_Pad_D1.5mm
- U16: footprint Package_TO_SOT_SMD:SOT-89-3 -> Xaar-Driver:SOT-89-3
Changed lines of the file:
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@@
-    )
-  )
-  (netclass_flag "" (length 2.54) (shape round) (at 105.41 86.36 90) (fields_autoplaced)
-    (effects (font (size 1.27 1.27)) (justify left bottom))
-    (property "Netclass" "HV" (at 102.87 85.6615 90)
-      (effects (font (size 1.27 1.27) italic) (justify left))
     )
   )
@@
       (effects (font (size 1.27 1.27)))
     )
-    (property "Footprint" "TestPoint:TestPoint_Pad_D1.5mm" (at 83.82 154.94 0)
+    (property "Footprint" "Xaar-Driver:TestPoint_Pad_D1.5mm" (at 83.82 154.94 0)
       (effects (font (size 1.27 1.27)) hide)
     )
@@
       (effects (font (size 1.27 1.27)) (justify right))
     )
-    (property "Footprint" "TestPoint:TestPoint_Pad_D1.5mm" (at 76.2 82.55 0)
+    (property "Footprint" "Xaar-Driver:TestPoint_Pad_D1.5mm" (at 76.2 82.55 0)
       (effects (font (size 1.27 1.27)) hide)
     )
@@
       (effects (font (size 1.27 1.27)) (justify right))
     )
-    (property "Footprint" "TestPoint:TestPoint_Pad_D1.5mm" (at 135.89 80.01 0)
+    (property "Footprint" "Xaar-Driver:TestPoint_Pad_D1.5mm" (at 135.89 80.01 0)
       (effects (font (size 1.27 1.27)) hide)
     )
@@
       (effects (font (size 1.27 1.27)))
     )
-    (property "Footprint" "TestPoint:TestPoint_Pad_D1.5mm" (at 134.62 140.97 0)
+    (property "Footprint" "Xaar-Driver:TestPoint_Pad_D1.5mm" (at 134.62 140.97 0)
       (effects (font (size 1.27 1.27)) hide)
     )
@@
       (effects (font (size 1.27 1.27)) (justify left))
     )
-    (property "Footprint" "TestPoint:TestPoint_Pad_D1.5mm" (at 92.71 165.1 0)
+    (property "Footprint" "Xaar-Driver:TestPoint_Pad_D1.5mm" (at 92.71 165.1 0)
       (effects (font (size 1.27 1.27)) hide)
     )
@@
       (effects (font (size 1.27 1.27)))
     )
-    (property "Footprint" "Package_TO_SOT_SMD:SOT-89-3" (at 100.33 38.1 0)
+    (property "Footprint" "Xaar-Driver:SOT-89-3" (at 100.33 38.1 0)
       (effects (font (size 1.27 1.27) italic) hide)
     )
@@
       (effects (font (size 1.27 1.27)))
     )
-    (property "Footprint" "TestPoint:TestPoint_Pad_D1.5mm" (at 201.93 44.45 0)
-      (effects (font (size 1.27 1.27)) hide)
-    )
+    (property "Footprint" "Xaar-Driver:TestPoint_Pad_D1.5mm" (at 201.93 44.45 0)
+      (effects (font (size 1.27 1.27)) hide)
+    )
