File: Xaar128-Driver/regulator.kicad_sch (KiCad schematic)
At the start: 42 parts, among them U11 LM317_TO-220, U13 MCP4725xxx-xCH, U14 ISO1540, U15 L7824, U16 MC78L05_SOT89, U17 TLC272, U18 MCP3021

Commit message: add acc and text
Parts:
- C21, C22, C23, C24, C26: value (none) -> 100n >16V Cer
Changed lines of the file:
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@@
       (effects (font (size 1.27 1.27)))
     )
-    (property "Value" "  " (at 66.04 130.81 90)
+    (property "Value" "100n >16V Cer" (at 66.04 130.81 90)
       (effects (font (size 1.27 1.27)))
     )
@@
       (effects (font (size 1.27 1.27)))
     )
-    (property "Value" "  " (at 78.74 64.77 90)
+    (property "Value" "100n >16V Cer" (at 78.74 64.77 90)
       (effects (font (size 1.27 1.27)))
     )
@@
       (effects (font (size 1.27 1.27)))
     )
-    (property "Value" "  " (at 175.26 121.92 90)
+    (property "Value" "100n >16V Cer" (at 175.26 121.92 90)
       (effects (font (size 1.27 1.27)))
     )
@@
       (effects (font (size 1.27 1.27)))
     )
-    (property "Value" "  " (at 119.38 62.23 90)
+    (property "Value" "100n >16V Cer" (at 119.38 62.23 90)
       (effects (font (size 1.27 1.27)))
     )
@@
       (effects (font (size 1.27 1.27)))
     )
-    (property "Value" "  " (at 44.45 130.81 90)
-      (effects (font (size 1.27 1.27)))
-    )
+    (property "Value" "100n >16V Cer" (at 44.45 130.81 90)
+      (effects (font (size 1.27 1.27)))
+    )

Commit message: ordering voltage regulator extension
Parts:
- C20, C21, C22, C23, C24, C25, C26, R33, R34, R35, R36, R41, R42, U13, U15, U16, U18: Extension (none) -> Regulator
- U14: value ISO1540 -> ISO1541; symbol Isolator:ISO1540 -> Isolator:ISO1541; Extension (none) -> Regulator; RSBestNr 825-3079 -> 825-3075
- U17: Extension (none) -> Regulator; Supplier Elekroplatz -> Elektroplatz
Changed lines of the file:
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@@
       (effects (font (size 1.27 1.27)) hide)
     )
-    (property "Supplier" "Elekroplatz" (at 125.73 80.01 0)
+    (property "Supplier" "Elektroplatz" (at 125.73 80.01 0)
+      (effects (font (size 1.27 1.27)) hide)
+    )
+    (property "Extension" "Regulator" (at 125.73 80.01 0)
       (effects (font (size 1.27 1.27)) hide)
     )
@@
       (effects (font (size 1.27 1.27)) hide)
     )
+    (property "Extension" "Regulator" (at 180.34 85.09 0)
+      (effects (font (size 1.27 1.27)) hide)
+    )
     (pin "1")
     (pin "2")
@@
       (effects (font (size 1.27 1.27)) hide)
     )
+    (property "Extension" "Regulator" (at 130.81 71.12 0)
+      (effects (font (size 1.27 1.27)) hide)
+    )
     (pin "1")
     (pin "2")
@@
     )
   )
-  (symbol (lib_id "Isolator:ISO1540") (at 52.07 151.13 0) (unit 1)
+  (symbol (lib_id "Isolator:ISO1541") (at 52.07 151.13 0) (unit 1)
     (in_bom yes) (on_board yes) (dnp yes)
     (property "Reference" "U14" (at 52.07 160.02 0)
       (effects (font (size 1.27 1.27)))
     )
-    (property "Value" "ISO1540" (at 52.07 162.56 0)
+    (property "Value" "ISO1541" (at 55.88 144.78 0)
       (effects (font (size 1.27 1.27)))
     )
@@
       (effects (font (size 1.27 1.27)) hide)
     )
-    (property "RSBestNr" "825-3079" (at 52.07 151.13 0)
+    (property "RSBestNr" "825-3075" (at 52.07 151.13 0)
       (effects (font (size 1.27 1.27)) hide)
     )
     (property "Supplier" "RS" (at 52.07 151.13 0)
+      (effects (font (size 1.27 1.27)) hide)
+    )
+    (property "Extension" "Regulator" (at 52.07 151.13 0)
       (effects (font (size 1.27 1.27)) hide)
     )
@@
       (effects (font (size 1.27 1.27)) hide)
     )
+    (property "Extension" "Regulator" (at 66.04 135.89 90)
+      (effects (font (size 1.27 1.27)) hide)
+    )
     (pin "1")
     (pin "2")
@@
     )
     (property "Supplier" "RS" (at 62.23 82.55 0)
+      (effects (font (size 1.27 1.27)) hide)
+    )
+    (property "Extension" "Regulator" (at 62.23 82.55 0)
       (effects (font (size 1.27 1.27)) hide)
     )
@@
       (effects (font (size 1.27 1.27)) hide)
     )
+    (property "Extension" "Regulator" (at 92.71 152.4 0)
+      (effects (font (size 1.27 1.27)) hide)
+    )
     (pin "1")
     (pin "2")
@@
       (effects (font (size 1.27 1.27)) hide)
     )
+    (property "Extension" "Regulator" (at 78.74 69.85 90)
+      (effects (font (size 1.27 1.27)) hide)
+    )
     (pin "1")
     (pin "2")
@@
     )
     (property "Supplier" "Elektroplatz" (at 157.48 80.01 0)
+      (effects (font (size 1.27 1.27)) hide)
+    )
+    (property "Extension" "Regulator" (at 157.48 80.01 0)
       (effects (font (size 1.27 1.27)) hide)
     )
@@
       (effects (font (size 1.27 1.27)) hide)
     )
+    (property "Extension" "Regulator" (at 109.22 77.47 0)
+      (effects (font (size 1.27 1.27)) hide)
+    )
     (pin "1")
     (pin "2")
@@
       (effects (font (size 1.27 1.27)) hide)
     )
+    (property "Extension" "Regulator" (at 175.26 125.73 90)
+      (effects (font (size 1.27 1.27)) hide)
+    )
     (pin "1")
     (pin "2")
@@
       (effects (font (size 1.27 1.27)) hide)
     )
-    (property "Supplier" "Elekroplatz" (at 123.19 80.01 0)
+    (property "Supplier" "Elektroplatz" (at 123.19 80.01 0)
+      (effects (font (size 1.27 1.27)) hide)
+    )
+    (property "Extension" "Regulator" (at 123.19 80.01 0)
       (effects (font (size 1.27 1.27)) hide)
     )
@@
       (effects (font (size 1.27 1.27)) hide)
     )
+    (property "Extension" "Regulator" (at 190.5 127.635 0)
+      (effects (font (size 1.27 1.27)) hide)
+    )
     (pin "1")
     (pin "2")
@@
       (effects (font (size 1.27 1.27)) hide)
     )
-    (property "Supplier" "Elekroplatz" (at 129.54 102.87 0)
+    (property "Supplier" "Elektroplatz" (at 129.54 102.87 0)
+      (effects (font (size 1.27 1.27)) hide)
+    )
+    (property "Extension" "Regulator" (at 129.54 102.87 0)
       (effects (font (size 1.27 1.27)) hide)
     )
@@
       (effects (font (size 1.27 1.27)) hide)
     )
+    (property "Extension" "Regulator" (at 175.26 132.08 90)
+      (effects (font (size 1.27 1.27)) hide)
+    )
     (pin "1")
     (pin "2")
@@
       (effects (font (size 1.27 1.27)) hide)
     )
+    (property "Extension" "Regulator" (at 119.38 67.31 90)
+      (effects (font (size 1.27 1.27)) hide)
+    )
     (pin "1")
     (pin "2")
@@
       (effects (font (size 1.27 1.27)) hide)
     )
+    (property "Extension" "Regulator" (at 134.62 135.89 0)
+      (effects (font (size 1.27 1.27)) hide)
+    )
     (pin "1")
     (pin "2")
@@
       (effects (font (size 1.27 1.27)) hide)
     )
+    (property "Extension" "Regulator" (at 44.45 135.89 90)
+      (effects (font (size 1.27 1.27)) hide)
+    )
     (pin "1")
     (pin "2")
@@
       (effects (font (size 1.27 1.27)) hide)
     )
+    (property "Extension" "Regulator" (at 149.86 33.02 0)
+      (effects (font (size 1.27 1.27)) hide)
+    )
     (pin "1")
     (pin "2")
@@
       (effects (font (size 1.27 1.27)) hide)
     )
+    (property "Extension" "Regulator" (at 100.33 33.02 0)
+      (effects (font (size 1.27 1.27)) hide)
+    )
     (pin "1")
     (pin "2")
@@
       (effects (font (size 1.27 1.27)) hide)
     )
+    (property "Extension" "Regulator" (at 31.75 143.51 0)
+      (effects (font (size 1.27 1.27)) hide)
+    )
     (pin "1")
     (pin "2")
@@
       (effects (font (size 1.27 1.27)) hide)
     )
+    (property "Extension" "Regulator" (at 68.58 73.66 90)
+      (effects (font (size 1.27 1.27)) hide)
+    )
     (pin "1")
     (pin "2")
@@
       (effects (font (size 1.27 1.27)) hide)
     )
+    (property "Extension" "Regulator" (at 35.56 143.51 0)
+      (effects (font (size 1.27 1.27)) hide)
+    )
     (pin "1")
     (pin "2")
@@
       (effects (font (size 1.27 1.27)) hide)
     )
+    (property "Extension" "Regulator" (at 134.62 154.94 0)
+      (effects (font (size 1.27 1.27)) hide)
+    )

Commit message: fix dac address r
Parts:
- added R60: 10k, Resistor_SMD:R_0603_1608Metric_Pad0.98x0.95mm_HandSolder, symbol Device:R
- renumbered D11 to D10, R33 to R30, R33 to R31, R33 to R32, R33 to R37, R33 to R38, R33 to R39, R33 to R40
Connections:
- net GND1: now also R60.2
- net at U13.6 (A0): now also R60.1
- no-connect marks 5 -> 4

Commit message: switch opv to lm358
Parts:
- U17: value TLC272 -> LM358; symbol Amplifier_Operational:TLC272 -> Amplifier_Operational:LM358
Changed lines of the file:
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@@
 	(wire
 		(pts
+			(xy 130.81 80.01) (xy 138.43 80.01)
+		)
+		(stroke
+			(width 0)
+			(type default)
+		)
+	)
+	(wire
+		(pts
 			(xy 158.75 33.02) (xy 161.29 33.02)
 		)
@@
 	(wire
 		(pts
-			(xy 130.81 80.01) (xy 138.43 80.01)
-		)
-		(stroke
-			(width 0)
-			(type default)
-		)
-	)
-	(wire
-		(pts
 			(xy 134.62 146.05) (xy 134.62 151.13)
 		)
@@
 	)
 	(symbol
-		(lib_id "Amplifier_Operational:TLC272")
+		(lib_id "Amplifier_Operational:LM358")
 		(at 125.73 80.01 0)
 		(unit 3)
@@
 			)
 		)
-		(property "Value" "TLC272"
-			(at 124.46 73.66 0)
+		(property "Value" "LM358"
+			(at 125.73 85.09 0)
 			(effects
 				(font
@@
 	)
 	(symbol
-		(lib_id "Amplifier_Operational:TLC272")
+		(lib_id "Amplifier_Operational:LM358")
 		(at 123.19 80.01 0)
 		(mirror x)
@@
 			)
 		)
-		(property "Value" "TLC272"
-			(at 129.54 83.82 0)
+		(property "Value" "LM358"
+			(at 123.19 74.93 0)
 			(effects
 				(font
 					(size 1.27 1.27)
 				)
+				(justify left)
 			)
 		)
@@
 	)
 	(symbol
-		(lib_id "Amplifier_Operational:TLC272")
+		(lib_id "Amplifier_Operational:LM358")
 		(at 129.54 102.87 0)
 		(unit 2)
@@
 			)
 		)
-		(property "Value" "TLC272"
+		(property "Value" "LM358"
 			(at 129.54 95.25 0)
 			(effects
