File: Xaar128-Driver/hv_supply.kicad_sch (KiCad schematic)
At the start: 18 parts, among them Q7 DMG2305UX, Q8 DMG2305UX, U19 LTV-356T

Commit message: 5v monitoring
Parts:
- added C7: 100n, symbol Device:C
- added D1: 3V, symbol Device:D_Zener
- added JP6: VPP_CHECK, symbol Jumper:Jumper_3_Bridged12
- added Q3 (x2): DMN2075U, Package_TO_SOT_SMD:SOT-23, symbol Transistor_FET:DMN2075U
- added R12, R13, R15, R16, R17 (x2): 10k, symbol Device:R
- added R14: 100k, symbol Device:R
- added R2: 2k, symbol Device:R
- added R3, R5: 1k, symbol Device:R
- added R59: 680, symbol Device:R
- added TP4: VPP_EN, symbol Connector:TestPoint
- added U3: 74HC173, symbol Xaar_Driver:74HC173
- R29: value 680 -> 1k
Connections:
- net GND: now also C7.2, Q3.2 (S), R13.2, R14.2, R15.2, R16.2, R17.2, R2.2, U3.8 (GND)
- net VPP_EN: now also R14.1, R3.1, R59.1; no longer R29.1
- net at R29.2: now also JP6.1 (A); no longer U19.1
- new net: R16.1, U3.10 (~{E2})
- new net: R17.1, U3.9 (~{E1})
- new net: R15.1, U3.1 (~{OE1})
- new net: R17.1, U3.14 (D0)
- new net: Q3.3 (D), R12.2, U3.15 (Mr)
- new net: R13.1, U3.2 (~{OE2})
- new net: R29.1, TP4.1, U3.3 (Q0)
- new net: Q3.1 (G), R3.2
- new net: Q3.2 (S), Q3.3 (D)
- new net: Q3.1 (G), R5.2
- new net: JP6.3 (B), R59.2
- new net: D1.2 (A), R2.1, R5.1
- new net: JP6.2 (C), U19.1
- new net +5V: C7.1, D1.1 (K), R12.1, R17.2, U3.16 (VCC)
- new net VPP_ENABLE_CP_5: U3.7 (Cp)
- no-connect marks 0 -> 6
Other:
- moved on the sheet: C11, C12, C13, C14, C15, C16, D1, D7, D8, F1, Q7, Q8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

Commit message: some component selections, fix wrong mcu
Parts:
- C11, C15, C16: value 1u -> 1u >72V Cer
- C12: value 10u -> 10u >72V E
- C13, C14: value 220u -> 220u >72V E
- C7: value 100n -> 100n >16V Cer; footprint (none) -> Capacitor_SMD:C_0603_1608Metric_Pad1.08x0.95mm_HandSolder; Supplier (none) -> Elektroplatz
- JP6: value VPP_CHECK -> Jumper_3_Bridged12; footprint (none) -> Connector_PinHeader_2.54mm:PinHeader_1x03_P2.54mm_Vertical; Funktion (none) -> Connect VPP_EN directly to MCU
- Q3: RSBestNr (none) -> 751-4143; Supplier (none) -> RS
- Q7, Q8: RSBestNr (none) -> 827-0452; Supplier (none) -> RS
- TP10: value U19_C -> TestPoint; footprint (none) -> TestPoint:TestPoint_Pad_D1.5mm; Funktion (none) -> U19_C; Supplier (none) -> None
- TP4: value VPP_EN -> TestPoint; footprint (none) -> TestPoint:TestPoint_Pad_D1.5mm; Funktion (none) -> VPP_EN; Supplier (none) -> None
- TP5: value Q7_8_Gate -> TestPoint; footprint (none) -> TestPoint:TestPoint_Pad_D1.5mm; Funktion (none) -> Q7_8_Gate; Supplier (none) -> None
- U19: RSBestNr (none) -> 691-2079; Supplier (none) -> RS

Commit message: assign footprints
Parts:
- C11, C15, C16: footprint (none) -> Capacitor_SMD:C_0805_2012Metric_Pad1.18x1.45mm_HandSolder; RSBestNr (none) -> 788-3054; Supplier (none) -> RS
- C12: footprint (none) -> Capacitor_SMD:CP_Elec_6.3x7.7; RSBestNr (none) -> 715-1442; Supplier (none) -> RS
- C13, C14: footprint (none) -> Capacitor_THT:CP_Radial_D13.0mm_P5.00mm; RSBestNr (none) -> 170-1289; Supplier (none) -> RS
- D1: value 5.6V -> 5.1V; footprint (none) -> Diode_THT:D_DO-35_SOD27_P7.62mm_Horizontal; Supplier (none) -> Elektroplatz
- D1: value 3V -> 3.3V; footprint (none) -> Diode_SMD:D_SOD-123F; RSBestNr (none) -> 792-0936; Supplier (none) -> RS
- D7, D8: value 1N4002 -> 1N4007; footprint (none) -> Diode_THT:D_DO-41_SOD81_P10.16mm_Horizontal; Supplier (none) -> Elektroplatz
- F1: footprint (none) -> FUSE_646_1_LTF:FUSE_646_1_LTF; Supplier (none) -> Printerbox
- JP6: Supplier (none) -> Elektroplatz
- R12, R13, R15, R16, R17: footprint (none) -> Resistor_SMD:R_0603_1608Metric_Pad0.98x0.95mm_HandSolder; Supplier (none) -> Elektroplatz
- R14: footprint (none) -> Resistor_SMD:R_0603_1608Metric_Pad0.98x0.95mm_HandSolder; RSBestNr (none) -> 678-9673; Supplier (none) -> RS
- R2: value 2k -> 2.2k; footprint (none) -> Resistor_SMD:R_0603_1608Metric_Pad0.98x0.95mm_HandSolder; Supplier (none) -> Elektroplatz
- R27: value 12k -> 12k > 200mW
- R29, R3, R5: footprint (none) -> Resistor_SMD:R_0603_1608Metric_Pad0.98x0.95mm_HandSolder; RSBestNr (none) -> 678-9875; Supplier (none) -> RS
- U3: footprint (none) -> Package_SO:SO-16_3.9x9.9mm_P1.27mm; RSBestNr (none) -> 483-6443; Supplier (none) -> RS

Commit message: select remaining components, nucleo footprint
Parts:
- C12: footprint Capacitor_SMD:CP_Elec_6.3x7.7 -> Capacitor_THT:CP_Radial_D5.0mm_P2.00mm; RSBestNr 715-1442 -> 228-7079
- C7: value 100n >16V Cer -> (none)
- R27: footprint (none) -> Resistor_SMD:R_1206_3216Metric_Pad1.30x1.75mm_HandSolder; RSBestNr (none) -> 812-1795; Supplier (none) -> RS
- R28: footprint (none) -> Resistor_SMD:R_0603_1608Metric_Pad0.98x0.95mm_HandSolder; RSBestNr (none) -> 198-5552; Supplier (none) -> RS
- R59: footprint (none) -> Resistor_SMD:R_0603_1608Metric_Pad0.98x0.95mm_HandSolder; RSBestNr (none) -> 679-0627; Supplier (none) -> RS
Changed lines of the file:
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@@
       (effects (font (size 1.27 1.27)) (justify right))
     )
-    (property "Footprint" "" (at 216.408 133.35 90)
+    (property "Footprint" "Resistor_SMD:R_0603_1608Metric_Pad0.98x0.95mm_HandSolder" (at 216.408 133.35 90)
       (effects (font (size 1.27 1.27)) hide)
     )
@@
       (effects (font (size 1.27 1.27)) hide)
     )
-    (property "RSBestNr" "" (at 214.63 133.35 0)
-      (effects (font (size 1.27 1.27)) hide)
-    )
-    (property "Supplier" "" (at 214.63 133.35 0)
+    (property "RSBestNr" "679-0627" (at 214.63 133.35 0)
+      (effects (font (size 1.27 1.27)) hide)
+    )
+    (property "Supplier" "RS" (at 214.63 133.35 0)
       (effects (font (size 1.27 1.27)) hide)
     )
@@
       (effects (font (size 1.27 1.27)) (justify left))
     )
-    (property "Footprint" "" (at 252.222 76.2 90)
+    (property "Footprint" "Resistor_SMD:R_0603_1608Metric_Pad0.98x0.95mm_HandSolder" (at 252.222 76.2 90)
       (effects (font (size 1.27 1.27)) hide)
     )
@@
       (effects (font (size 1.27 1.27)) hide)
     )
-    (property "RSBestNr" "" (at 254 76.2 0)
-      (effects (font (size 1.27 1.27)) hide)
-    )
-    (property "Supplier" "" (at 254 76.2 0)
+    (property "RSBestNr" "198-5552" (at 254 76.2 0)
+      (effects (font (size 1.27 1.27)) hide)
+    )
+    (property "Supplier" "RS" (at 254 76.2 0)
       (effects (font (size 1.27 1.27)) hide)
     )
@@
       (effects (font (size 1.27 1.27)))
     )
-    (property "Value" "100n >16V Cer" (at 158.75 102.87 90)
+    (property "Value" "  " (at 158.75 102.87 90)
       (effects (font (size 1.27 1.27)))
     )
@@
       (effects (font (size 1.27 1.27)) (justify left))
     )
-    (property "Footprint" "Capacitor_SMD:CP_Elec_6.3x7.7" (at 225.7552 72.39 0)
+    (property "Footprint" "Capacitor_THT:CP_Radial_D5.0mm_P2.00mm" (at 225.7552 72.39 0)
       (effects (font (size 1.27 1.27)) hide)
     )
@@
       (effects (font (size 1.27 1.27)) hide)
     )
-    (property "RSBestNr" "715-1442" (at 224.79 68.58 0)
+    (property "RSBestNr" "228-7079" (at 224.79 68.58 0)
       (effects (font (size 1.27 1.27)) hide)
     )
@@
       (effects (font (size 1.27 1.27)) (justify left))
     )
-    (property "Footprint" "" (at 243.332 99.06 90)
+    (property "Footprint" "Resistor_SMD:R_1206_3216Metric_Pad1.30x1.75mm_HandSolder" (at 243.332 99.06 90)
       (effects (font (size 1.27 1.27)) hide)
     )
@@
       (effects (font (size 1.27 1.27)) hide)
     )
-    (property "RSBestNr" "" (at 245.11 99.06 0)
-      (effects (font (size 1.27 1.27)) hide)
-    )
-    (property "Supplier" "" (at 245.11 99.06 0)
-      (effects (font (size 1.27 1.27)) hide)
-    )
+    (property "RSBestNr" "812-1795" (at 245.11 99.06 0)
+      (effects (font (size 1.27 1.27)) hide)
+    )
+    (property "Supplier" "RS" (at 245.11 99.06 0)
+      (effects (font (size 1.27 1.27)) hide)
+    )

Commit message: xaar driver: some routed islands
Connections:
- net GNDHP is gone; now on net GND1: C13.2, C14.2, C16.2
Changed lines of the file:
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@@
     )
   )
-  (symbol (lib_id "Xaar_Driver:GNDHP") (at 177.8 78.74 0) (unit 1)
+  (symbol (lib_id "power:GND1") (at 177.8 78.74 0) (unit 1)
     (in_bom yes) (on_board yes) (dnp no) (fields_autoplaced)
-    (property "Reference" "#PWR0100" (at 177.8 85.09 0)
+    (property "Reference" "#PWR0113" (at 177.8 85.09 0)
       (effects (font (size 1.27 1.27)) hide)
     )
-    (property "Value" "GNDHP" (at 177.8 83.82 0)
+    (property "Value" "GND1" (at 177.8 83.82 0)
       (effects (font (size 1.27 1.27)))
     )
@@
       (project "Xaar128-Driver"
         (path "/f0c82013-03f9-4093-aa02-30b89fd69529/1b3c0a7f-2f11-4b02-93de-b1cd5fa046f0"
-          (reference "#PWR0100") (unit 1)
+          (reference "#PWR0113") (unit 1)
         )
       )

Commit message: almost
Parts:
- D8: footprint Diode_THT:D_DO-41_SOD81_P10.16mm_Horizontal -> Diode_THT:D_DO-41_SOD81_P12.70mm_Horizontal
Changed lines of the file:
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@@
       (effects (font (size 1.27 1.27)))
     )
-    (property "Footprint" "Diode_THT:D_DO-41_SOD81_P10.16mm_Horizontal" (at 213.36 43.18 0)
+    (property "Footprint" "Diode_THT:D_DO-41_SOD81_P12.70mm_Horizontal" (at 213.36 43.18 0)
       (effects (font (size 1.27 1.27)) hide)
     )

Commit message: drc & plots done
Parts:
- TP10, TP4, TP5: footprint TestPoint:TestPoint_Pad_D1.5mm -> Xaar-Driver:TestPoint_Pad_D1.5mm
Changed lines of the file:
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@@
       (effects (font (size 1.27 1.27)) (justify left))
     )
-    (property "Footprint" "TestPoint:TestPoint_Pad_D1.5mm" (at 245.11 124.46 0)
+    (property "Footprint" "Xaar-Driver:TestPoint_Pad_D1.5mm" (at 245.11 124.46 0)
       (effects (font (size 1.27 1.27)) hide)
     )
@@
       (effects (font (size 1.27 1.27)) (justify right))
     )
-    (property "Footprint" "TestPoint:TestPoint_Pad_D1.5mm" (at 168.91 119.38 0)
+    (property "Footprint" "Xaar-Driver:TestPoint_Pad_D1.5mm" (at 168.91 119.38 0)
       (effects (font (size 1.27 1.27)) hide)
     )
@@
       (effects (font (size 1.27 1.27)) (justify right))
     )
-    (property "Footprint" "TestPoint:TestPoint_Pad_D1.5mm" (at 193.04 91.44 0)
-      (effects (font (size 1.27 1.27)) hide)
-    )
+    (property "Footprint" "Xaar-Driver:TestPoint_Pad_D1.5mm" (at 193.04 91.44 0)
+      (effects (font (size 1.27 1.27)) hide)
+    )

Commit message: add acc and text
Parts:
- C7: value (none) -> 100n >16V Cer
Changed lines of the file:
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@@
       (effects (font (size 1.27 1.27)))
     )
-    (property "Value" "  " (at 158.75 102.87 90)
+    (property "Value" "100n >16V Cer" (at 158.75 102.87 90)
       (effects (font (size 1.27 1.27)))
     )
