File: Xaar128-Driver/hv_supply.kicad_sch (KiCad schematic)
At the start: 36 parts, among them Q3 DMN2075U, Q7 DMG2305UX, Q8 DMG2305UX, U19 LTV-356T, U3 74HC173

Commit message: fix caps
Parts:
- C13, C14: RSBestNr 170-1289 -> 711-1734
Changed lines of the file:
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@@
       (effects (font (size 1.27 1.27)) hide)
     )
-    (property "RSBestNr" "170-1289" (at 165.1 68.58 0)
+    (property "RSBestNr" "711-1734" (at 165.1 68.58 0)
       (effects (font (size 1.27 1.27)) hide)
     )
@@
       (effects (font (size 1.27 1.27)) hide)
     )
-    (property "RSBestNr" "170-1289" (at 177.8 68.58 0)
-      (effects (font (size 1.27 1.27)) hide)
-    )
+    (property "RSBestNr" "711-1734" (at 177.8 68.58 0)
+      (effects (font (size 1.27 1.27)) hide)
+    )

Commit message: create order list
Parts:
- R28: footprint Resistor_SMD:R_0603_1608Metric_Pad0.98x0.95mm_HandSolder -> Resistor_SMD:R_0805_2012Metric_Pad1.20x1.40mm_HandSolder; RSBestNr 198-5552 -> 721-7804
Changed lines of the file:
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@@
       (effects (font (size 1.27 1.27)) (justify left))
     )
-    (property "Footprint" "Resistor_SMD:R_0603_1608Metric_Pad0.98x0.95mm_HandSolder" (at 252.222 76.2 90)
+    (property "Footprint" "Resistor_SMD:R_0805_2012Metric_Pad1.20x1.40mm_HandSolder" (at 252.222 76.2 90)
       (effects (font (size 1.27 1.27)) hide)
     )
@@
       (effects (font (size 1.27 1.27)) hide)
     )
-    (property "RSBestNr" "198-5552" (at 254 76.2 0)
+    (property "RSBestNr" "721-7804" (at 254 76.2 0)
       (effects (font (size 1.27 1.27)) hide)
     )

Commit message: fix dac address r
Parts:
- renumbered C7 to C31, D1 to D5, D1 to D9, JP6 to JP14, Q3 to Q4, Q3 to Q5, R16 to R21, R17 to R44, R17 to R50, R13 to R51, R15 to R52, R12 to R54, R3 to R55, R14 to R56, R2 to R57, R5 to R58, TP4 to TP13, U3 to U21

Commit message: correct pmos
Parts:
- Q7, Q8: value DMG2305UX -> SI2319CDS-T1-GE3; RSBestNr 827-0452 -> 787-9042
Changed lines of the file:
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@@
 			)
 		)
-		(property "Value" "DMG2305UX"
+		(property "Value" "SI2319CDS-T1-GE3"
 			(at 267.97 90.17 0)
 			(effects
@@
 			)
 		)
-		(property "Datasheet" "https://www.diodes.com/assets/Datasheets/DMG2301L.pdf"
+		(property "Datasheet" ""
 			(at 261.62 91.44 0)
 			(effects
@@
 			)
 		)
-		(property "RSBestNr" "827-0452"
+		(property "RSBestNr" "787-9042"
 			(at 261.62 91.44 0)
 			(effects
@@
 			)
 		)
-		(property "Value" "DMG2305UX"
+		(property "Value" "SI2319CDS-T1-GE3"
 			(at 129.54 90.17 0)
 			(effects
@@
 			)
 		)
-		(property "Datasheet" "https://www.diodes.com/assets/Datasheets/DMG2301L.pdf"
+		(property "Datasheet" ""
 			(at 135.89 91.44 0)
 			(effects
@@
 			)
 		)
-		(property "RSBestNr" "827-0452"
+		(property "RSBestNr" "787-9042"
 			(at 135.89 91.44 0)
 			(effects
