File: Xaar128-Driver/mcu.kicad_sch (KiCad schematic)
At the start: 11 parts, among them U4 NUCLEO-H743ZI2

Commit message: more routing
Connections:
- net VPP_ENABLE_CP: now also U4.11 (PC3); no longer U4.13 (PC2)
- net nRESET_MCU: now also U4.13 (PC2); no longer U4.11 (PC3)
Changed lines of the file:
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@@
     (effects (font (size 1.27 1.27)) (justify left bottom))
+  )
+  (hierarchical_label "VPP_ENABLE_CP" (shape output) (at 113.03 90.17 180) (fields_autoplaced)
+    (effects (font (size 1.27 1.27)) (justify right))
   )
   (hierarchical_label "MOSI" (shape output) (at 212.09 68.58 0) (fields_autoplaced)
@@
   (hierarchical_label "nSS1" (shape output) (at 212.09 88.9 0) (fields_autoplaced)
     (effects (font (size 1.27 1.27)) (justify left))
+  )
+  (hierarchical_label "RESET_DISABLE_CP" (shape output) (at 113.03 87.63 180) (fields_autoplaced)
+    (effects (font (size 1.27 1.27)) (justify right))
   )
   (hierarchical_label "PHO" (shape output) (at 134.62 149.86 270) (fields_autoplaced)
@@
     (effects (font (size 1.27 1.27)) (justify left))
   )
-  (hierarchical_label "RESET_DISABLE_CP" (shape output) (at 113.03 87.63 180) (fields_autoplaced)
-    (effects (font (size 1.27 1.27)) (justify right))
-  )
   (hierarchical_label "SDA" (shape output) (at 212.09 55.88 0) (fields_autoplaced)
     (effects (font (size 1.27 1.27)) (justify left))
@@
     (effects (font (size 1.27 1.27)) (justify left))
   )
-  (hierarchical_label "VPP_ENABLE_CP" (shape output) (at 113.03 95.25 180) (fields_autoplaced)
-    (effects (font (size 1.27 1.27)) (justify right))
-  )
   (hierarchical_label "nRESET_IN" (shape input) (at 113.03 92.71 180) (fields_autoplaced)
-    (effects (font (size 1.27 1.27)) (justify right))
-  )
-  (hierarchical_label "nRESET_MCU" (shape output) (at 113.03 90.17 180) (fields_autoplaced)
     (effects (font (size 1.27 1.27)) (justify right))
   )
@@
     (effects (font (size 1.27 1.27)) (justify left))
   )
+  (hierarchical_label "nRESET_MCU" (shape output) (at 113.03 95.25 180) (fields_autoplaced)
+    (effects (font (size 1.27 1.27)) (justify right))
+  )
   (hierarchical_label "VPP_EN" (shape output) (at 142.24 135.89 270) (fields_autoplaced)

Commit message: create order list
Parts:
- JP10, JP11, JP16: RSBestNr 120-432 -> (none); Supplier RS -> None
- JP13, JP3: RSBestNr 120-432 -> 820-6736
- JP15, JP8, JP9: RSBestNr (none) -> 820-6736; Supplier None -> RS
Changed lines of the file:
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@@
       (effects (font (size 1.27 1.27)) hide)
     )
-    (property "RSBestNr" "120-432" (at 142.24 116.84 0)
-      (effects (font (size 1.27 1.27)) hide)
-    )
-    (property "Supplier" "RS" (at 142.24 116.84 0)
+    (property "RSBestNr" "" (at 142.24 116.84 0)
+      (effects (font (size 1.27 1.27)) hide)
+    )
+    (property "Supplier" "None" (at 142.24 116.84 0)
       (effects (font (size 1.27 1.27)) hide)
     )
@@
       (effects (font (size 1.27 1.27)) hide)
     )
-    (property "RSBestNr" "120-432" (at 147.32 116.84 0)
-      (effects (font (size 1.27 1.27)) hide)
-    )
-    (property "Supplier" "RS" (at 147.32 116.84 0)
+    (property "RSBestNr" "" (at 147.32 116.84 0)
+      (effects (font (size 1.27 1.27)) hide)
+    )
+    (property "Supplier" "None" (at 147.32 116.84 0)
       (effects (font (size 1.27 1.27)) hide)
     )
@@
       (effects (font (size 1.27 1.27)) hide)
     )
-    (property "RSBestNr" "" (at 198.12 93.98 0)
-      (effects (font (size 1.27 1.27)) hide)
-    )
-    (property "Supplier" "None" (at 198.12 93.98 0)
+    (property "RSBestNr" "820-6736" (at 198.12 93.98 0)
+      (effects (font (size 1.27 1.27)) hide)
+    )
+    (property "Supplier" "RS" (at 198.12 93.98 0)
       (effects (font (size 1.27 1.27)) hide)
     )
@@
       (effects (font (size 1.27 1.27)) hide)
     )
-    (property "RSBestNr" "" (at 198.12 68.58 0)
-      (effects (font (size 1.27 1.27)) hide)
-    )
-    (property "Supplier" "None" (at 198.12 68.58 0)
+    (property "RSBestNr" "820-6736" (at 198.12 68.58 0)
+      (effects (font (size 1.27 1.27)) hide)
+    )
+    (property "Supplier" "RS" (at 198.12 68.58 0)
       (effects (font (size 1.27 1.27)) hide)
     )
@@
       (effects (font (size 1.27 1.27)) hide)
     )
-    (property "RSBestNr" "120-432" (at 149.86 116.84 0)
-      (effects (font (size 1.27 1.27)) hide)
-    )
-    (property "Supplier" "RS" (at 149.86 116.84 0)
+    (property "RSBestNr" "" (at 149.86 116.84 0)
+      (effects (font (size 1.27 1.27)) hide)
+    )
+    (property "Supplier" "None" (at 149.86 116.84 0)
       (effects (font (size 1.27 1.27)) hide)
     )
@@
       (effects (font (size 1.27 1.27)) hide)
     )
-    (property "RSBestNr" "" (at 198.12 63.5 0)
-      (effects (font (size 1.27 1.27)) hide)
-    )
-    (property "Supplier" "None" (at 198.12 63.5 0)
+    (property "RSBestNr" "820-6736" (at 198.12 63.5 0)
+      (effects (font (size 1.27 1.27)) hide)
+    )
+    (property "Supplier" "RS" (at 198.12 63.5 0)
       (effects (font (size 1.27 1.27)) hide)
     )
@@
       (effects (font (size 1.27 1.27)) hide)
     )
-    (property "RSBestNr" "120-432" (at 198.12 73.66 0)
+    (property "RSBestNr" "820-6736" (at 198.12 73.66 0)
       (effects (font (size 1.27 1.27)) hide)
     )
@@
       (effects (font (size 1.27 1.27)) hide)
     )
-    (property "RSBestNr" "120-432" (at 134.62 139.7 0)
-      (effects (font (size 1.27 1.27)) hide)
-    )
+    (property "RSBestNr" "820-6736" (at 134.62 139.7 0)
+      (effects (font (size 1.27 1.27)) hide)
+    )
