File: Xaar128-Driver/mcu.kicad_sch (KiCad schematic)
At the start: 11 parts, among them U4 NUCLEO-H743ZI2

Commit message: switch mcu
Parts:
- U4: symbol Xaar_Driver:NUCLEO-H743-Arduino -> Xaar_Driver:NUCLEO-H7A3-Arduino; RSBestNr 193-9787 -> 198-8645
Changed lines of the file:
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@@
     )
   )
-  (symbol (lib_id "Xaar_Driver:NUCLEO-H743-Arduino") (at 140.97 73.66 0) (unit 1)
+  (symbol (lib_id "Xaar_Driver:NUCLEO-H7A3-Arduino") (at 140.97 73.66 0) (unit 1)
     (in_bom yes) (on_board yes) (dnp no) (fields_autoplaced)
     (property "Reference" "U4" (at 155.3131 41.91 0)
@@
       (effects (font (size 1.27 1.27)) hide)
     )
-    (property "RSBestNr" "193-9787" (at 140.97 73.66 0)
+    (property "RSBestNr" "198-8645" (at 140.97 73.66 0)
       (effects (font (size 1.27 1.27)) hide)
     )
