File: Xaar128-Driver/io.kicad_sch (KiCad schematic)
At the start: 4 parts, among them J1 Screw_Terminal_01x02, J3 Screw_Terminal_01x02, J4 Screw_Terminal_01x02, J7 Screw_Terminal_01x04

Commit message: drc & plots done
Parts:
- removed J7: Screw_Terminal_01x04, RS_PRO:Steckbarer_Klemmenblock_1x04_5.08mm_vertical_copy, symbol Connector:Screw_Terminal_01x04
- added H1, H2, H3, H4: MountingHole, MountingHole:MountingHole_2.7mm_M2.5_DIN965, symbol Mechanical:MountingHole
- added J2, J7: Screw_Terminal_01x02, RS_PRO:897-1051, symbol Connector:Screw_Terminal_01x02
- J1, J3, J4: footprint RS_PRO:Steckbarer_Klemmenblock_1x02_5.08mm_vertical -> RS_PRO:897-1051; RSBestNr 897-1238 -> 897-1051 + 897-0998
Connections:
- net GND: now also J2.2 (Pin_2)
- net LED+: now also J7.2 (Pin_2)
- net LED-: now also J2.1 (Pin_1)
- net LED_PWR: now also J7.1 (Pin_1)
Changed lines of the file:
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@@
-    )
-  )
-  (netclass_flag "" (length 2.54) (shape round) (at 116.84 118.11 180) (fields_autoplaced)
-    (effects (font (size 1.27 1.27)) (justify right bottom))
-    (property "Netclass" "HV" (at 117.5385 120.65 0)
-      (effects (font (size 1.27 1.27) italic) (justify left))
     )
   )
@@
     )
   )
-  (symbol (lib_id "Connector:Screw_Terminal_01x04") (at 144.78 88.9 0) (unit 1)
-    (in_bom yes) (on_board yes) (dnp no) (fields_autoplaced)
-    (property "Reference" "J7" (at 147.32 88.9 0)
-      (effects (font (size 1.27 1.27)) (justify left))
-    )
-    (property "Value" "Screw_Terminal_01x04" (at 147.32 91.44 0)
-      (effects (font (size 1.27 1.27)) (justify left))
-    )
-    (property "Footprint" "RS_PRO:Steckbarer_Klemmenblock_1x04_5.08mm_vertical_copy" (at 144.78 88.9 0)
-      (effects (font (size 1.27 1.27)) hide)
-    )
-    (property "Datasheet" "~" (at 144.78 88.9 0)
-      (effects (font (size 1.27 1.27)) hide)
-    )
-    (property "RSBestNr" "897-1240" (at 144.78 88.9 0)
-      (effects (font (size 1.27 1.27)) hide)
-    )
-    (property "Supplier" "RS" (at 144.78 88.9 0)
-      (effects (font (size 1.27 1.27)) hide)
-    )
-    (pin "1")
-    (pin "2")
-    (pin "3")
-    (pin "4")
-    (instances
-      (project "Xaar128-Driver"
-        (path "/f0c82013-03f9-4093-aa02-30b89fd69529/8d2d865b-5c5b-48bf-9eef-a5e158c4d497"
-          (reference "J7") (unit 1)
-        )
-      )
-    )
-  )
   (symbol (lib_id "power:GND") (at 135.89 130.81 270) (unit 1)
     (in_bom yes) (on_board yes) (dnp no) (fields_autoplaced)
@@
     )
   )
+  (symbol (lib_id "Mechanical:MountingHole") (at 106.68 59.69 0) (unit 1)
+    (in_bom yes) (on_board yes) (dnp no) (fields_autoplaced)
+    (property "Reference" "H2" (at 109.22 58.42 0)
+      (effects (font (size 1.27 1.27)) (justify left))
+    )
+    (property "Value" "MountingHole" (at 109.22 60.96 0)
+      (effects (font (size 1.27 1.27)) (justify left))
+    )
+    (property "Footprint" "MountingHole:MountingHole_2.7mm_M2.5_DIN965" (at 106.68 59.69 0)
+      (effects (font (size 1.27 1.27)) hide)
+    )
+    (property "Datasheet" "~" (at 106.68 59.69 0)
+      (effects (font (size 1.27 1.27)) hide)
+    )
+    (instances
+      (project "Xaar128-Driver"
+        (path "/f0c82013-03f9-4093-aa02-30b89fd69529/8d2d865b-5c5b-48bf-9eef-a5e158c4d497"
+          (reference "H2") (unit 1)
+        )
+      )
+    )
+  )
+  (symbol (lib_id "Mechanical:MountingHole") (at 106.68 64.77 0) (unit 1)
+    (in_bom yes) (on_board yes) (dnp no) (fields_autoplaced)
+    (property "Reference" "H3" (at 109.22 63.5 0)
+      (effects (font (size 1.27 1.27)) (justify left))
+    )
+    (property "Value" "MountingHole" (at 109.22 66.04 0)
+      (effects (font (size 1.27 1.27)) (justify left))
+    )
+    (property "Footprint" "MountingHole:MountingHole_2.7mm_M2.5_DIN965" (at 106.68 64.77 0)
+      (effects (font (size 1.27 1.27)) hide)
+    )
+    (property "Datasheet" "~" (at 106.68 64.77 0)
+      (effects (font (size 1.27 1.27)) hide)
+    )
+    (instances
+      (project "Xaar128-Driver"
+        (path "/f0c82013-03f9-4093-aa02-30b89fd69529/8d2d865b-5c5b-48bf-9eef-a5e158c4d497"
+          (reference "H3") (unit 1)
+        )
+      )
+    )
+  )
   (symbol (lib_id "Connector:Screw_Terminal_01x02") (at 144.78 128.27 0) (unit 1)
     (in_bom yes) (on_board yes) (dnp no) (fields_autoplaced)
@@
       (effects (font (size 1.27 1.27)) (justify left))
     )
-    (property "Footprint" "RS_PRO:Steckbarer_Klemmenblock_1x02_5.08mm_vertical" (at 144.78 128.27 0)
+    (property "Footprint" "RS_PRO:897-1051" (at 144.78 128.27 0)
       (effects (font (size 1.27 1.27)) hide)
     )
@@
       (effects (font (size 1.27 1.27)) hide)
     )
-    (property "RSBestNr" "897-1238" (at 144.78 128.27 0)
+    (property "RSBestNr" "897-1051 + 897-0998" (at 144.78 128.27 0)
       (effects (font (size 1.27 1.27)) hide)
     )
@@
       (effects (font (size 1.27 1.27)) (justify left))
     )
-    (property "Footprint" "RS_PRO:Steckbarer_Klemmenblock_1x02_5.08mm_vertical" (at 144.78 99.06 0)
+    (property "Footprint" "RS_PRO:897-1051" (at 144.78 99.06 0)
       (effects (font (size 1.27 1.27)) hide)
     )
@@
       (effects (font (size 1.27 1.27)) hide)
     )
-    (property "RSBestNr" "897-1238" (at 144.78 99.06 0)
+    (property "RSBestNr" "897-1051 + 897-0998" (at 144.78 99.06 0)
       (effects (font (size 1.27 1.27)) hide)
     )
@@
       (effects (font (size 1.27 1.27)) (justify left))
     )
-    (property "Footprint" "RS_PRO:Steckbarer_Klemmenblock_1x02_5.08mm_vertical" (at 144.78 115.57 0)
+    (property "Footprint" "RS_PRO:897-1051" (at 144.78 115.57 0)
       (effects (font (size 1.27 1.27)) hide)
     )
@@
       (effects (font (size 1.27 1.27)) hide)
     )
-    (property "RSBestNr" "897-1238" (at 144.78 115.57 0)
+    (property "RSBestNr" "897-1051 + 897-0998" (at 144.78 115.57 0)
       (effects (font (size 1.27 1.27)) hide)
     )
@@
     )
   )
+  (symbol (lib_id "Mechanical:MountingHole") (at 106.68 69.85 0) (unit 1)
+    (in_bom yes) (on_board yes) (dnp no) (fields_autoplaced)
+    (property "Reference" "H4" (at 109.22 68.58 0)
+      (effects (font (size 1.27 1.27)) (justify left))
+    )
+    (property "Value" "MountingHole" (at 109.22 71.12 0)
+      (effects (font (size 1.27 1.27)) (justify left))
+    )
+    (property "Footprint" "MountingHole:MountingHole_2.7mm_M2.5_DIN965" (at 106.68 69.85 0)
+      (effects (font (size 1.27 1.27)) hide)
+    )
+    (property "Datasheet" "~" (at 106.68 69.85 0)
+      (effects (font (size 1.27 1.27)) hide)
+    )
+    (instances
+      (project "Xaar128-Driver"
+        (path "/f0c82013-03f9-4093-aa02-30b89fd69529/8d2d865b-5c5b-48bf-9eef-a5e158c4d497"
+          (reference "H4") (unit 1)
+        )
+      )
+    )
+  )
+  (symbol (lib_id "Connector:Screw_Terminal_01x02") (at 144.78 86.36 0) (unit 1)
+    (in_bom yes) (on_board yes) (dnp no) (fields_autoplaced)
+    (property "Reference" "J7" (at 147.32 86.36 0)
+      (effects (font (size 1.27 1.27)) (justify left))
+    )
+    (property "Value" "Screw_Terminal_01x02" (at 147.32 88.9 0)
+      (effects (font (size 1.27 1.27)) (justify left))
+    )
+    (property "Footprint" "RS_PRO:897-1051" (at 144.78 86.36 0)
+      (effects (font (size 1.27 1.27)) hide)
+    )
+    (property "Datasheet" "~" (at 144.78 86.36 0)
+      (effects (font (size 1.27 1.27)) hide)
+    )
+    (property "RSBestNr" "897-1051 + 897-0998" (at 144.78 86.36 0)
+      (effects (font (size 1.27 1.27)) hide)
+    )
+    (property "Supplier" "RS" (at 144.78 86.36 0)
+      (effects (font (size 1.27 1.27)) hide)
+    )
+    (pin "1")
+    (pin "2")
+    (instances
+      (project "Xaar128-Driver"
+        (path "/f0c82013-03f9-4093-aa02-30b89fd69529/8d2d865b-5c5b-48bf-9eef-a5e158c4d497"
+          (reference "J7") (unit 1)
+        )
+      )
+    )
+  )
+  (symbol (lib_id "Mechanical:MountingHole") (at 106.68 54.61 0) (unit 1)
+    (in_bom yes) (on_board yes) (dnp no) (fields_autoplaced)
+    (property "Reference" "H1" (at 109.22 53.34 0)
+      (effects (font (size 1.27 1.27)) (justify left))
+    )
+    (property "Value" "MountingHole" (at 109.22 55.88 0)
+      (effects (font (size 1.27 1.27)) (justify left))
+    )
+    (property "Footprint" "MountingHole:MountingHole_2.7mm_M2.5_DIN965" (at 106.68 54.61 0)
+      (effects (font (size 1.27 1.27)) hide)
+    )
+    (property "Datasheet" "~" (at 106.68 54.61 0)
+      (effects (font (size 1.27 1.27)) hide)
+    )
+    (instances
+      (project "Xaar128-Driver"
+        (path "/f0c82013-03f9-4093-aa02-30b89fd69529/8d2d865b-5c5b-48bf-9eef-a5e158c4d497"
+          (reference "H1") (unit 1)
+        )
+      )
+    )
+  )
   (symbol (lib_id "power:PWR_FLAG") (at 135.89 115.57 0) (unit 1)
     (in_bom yes) (on_board yes) (dnp no) (fields_autoplaced)
@@
         )
       )
+    )
+  )
+  (symbol (lib_id "Connector:Screw_Terminal_01x02") (at 144.78 91.44 0) (unit 1)
+    (in_bom yes) (on_board yes) (dnp no) (fields_autoplaced)
+    (property "Reference" "J2" (at 147.32 91.44 0)
+      (effects (font (size 1.27 1.27)) (justify left))
+    )
+    (property "Value" "Screw_Terminal_01x02" (at 147.32 93.98 0)
+      (effects (font (size 1.27 1.27)) (justify left))
+    )
+    (property "Footprint" "RS_PRO:897-1051" (at 144.78 91.44 0)
+      (effects (font (size 1.27 1.27)) hide)
+    )
+    (property "Datasheet" "~" (at 144.78 91.44 0)
+      (effects (font (size 1.27 1.27)) hide)
+    )
+    (property "RSBestNr" "897-1051 + 897-0998" (at 144.78 91.44 0)
+      (effects (font (size 1.27 1.27)) hide)
+    )
+    (property "Supplier" "RS" (at 144.78 91.44 0)
+      (effects (font (size 1.27 1.27)) hide)
+    )
+    (pin "1")
+    (pin "2")
+    (instances
+      (project "Xaar128-Driver"
+        (path "/f0c82013-03f9-4093-aa02-30b89fd69529/8d2d865b-5c5b-48bf-9eef-a5e158c4d497"
+          (reference "J2") (unit 1)
+        )
+      )

Commit message: create order list
Parts:
- H1, H2, H3, H4: Supplier (none) -> None
Changed lines of the file:
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@@
+      (effects (font (size 1.27 1.27)) hide)
+    )
+    (property "Supplier" "None" (at 106.68 59.69 0)
       (effects (font (size 1.27 1.27)) hide)
     )
@@
     )
     (property "Datasheet" "~" (at 106.68 64.77 0)
+      (effects (font (size 1.27 1.27)) hide)
+    )
+    (property "Supplier" "None" (at 106.68 64.77 0)
       (effects (font (size 1.27 1.27)) hide)
     )
@@
       (effects (font (size 1.27 1.27)) hide)
     )
+    (property "Supplier" "None" (at 106.68 69.85 0)
+      (effects (font (size 1.27 1.27)) hide)
+    )
     (instances
       (project "Xaar128-Driver"
@@
       (effects (font (size 1.27 1.27)) hide)
     )
+    (property "Supplier" "None" (at 106.68 54.61 0)
+      (effects (font (size 1.27 1.27)) hide)
+    )
