File: Xaar128-Driver/Xaar128-Driver.kicad_sch (KiCad schematic)
At the start: 0 parts

Commit message: 5v monitoring
Other:
- sheet HV Supply ports: added VPP_ENABLE_CP_5; removed none
- sheet Level Shift ports: added VPP_EN_CP_IN, VPP_EN_CP_OUT; removed none
- sheet MCU ports: added VPP_ENABLE_CP; removed none

Commit message: add acc and text
Other:
- added sheet ACC (acc.kicad_sch)
Changed lines of the file:
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@@
   (junction (at 190.5 106.68) (diameter 0) (color 0 0 0 0)
   )
+  (junction (at 87.63 45.72) (diameter 0) (color 0 0 0 0)
+  )
   (junction (at 189.23 40.64) (diameter 0) (color 0 0 0 0)
   )
+  (junction (at 93.98 48.26) (diameter 0) (color 0 0 0 0)
+  )
   (wire (pts (xy 190.5 81.28) (xy 185.42 81.28))
     (stroke (width 0) (type default))
@@
     (stroke (width 0) (type default))
   )
+  (wire (pts (xy 104.14 66.04) (xy 93.98 66.04))
+    (stroke (width 0) (type default))
+  )
   (wire (pts (xy 76.2 116.84) (xy 96.52 116.84))
     (stroke (width 0) (type default))
@@
     (stroke (width 0) (type default))
   )
+  (wire (pts (xy 87.63 45.72) (xy 104.14 45.72))
+    (stroke (width 0) (type default))
+  )
   (wire (pts (xy 147.32 99.06) (xy 151.13 99.06))
     (stroke (width 0) (type default))
   )
+  (wire (pts (xy 93.98 48.26) (xy 104.14 48.26))
+    (stroke (width 0) (type default))
+  )
   (wire (pts (xy 147.32 101.6) (xy 231.14 101.6))
     (stroke (width 0) (type default))
@@
     (stroke (width 0) (type default))
   )
-  (wire (pts (xy 76.2 45.72) (xy 104.14 45.72))
+  (wire (pts (xy 76.2 45.72) (xy 87.63 45.72))
     (stroke (width 0) (type default))
   )
@@
     (stroke (width 0) (type default))
   )
+  (wire (pts (xy 104.14 63.5) (xy 87.63 63.5))
+    (stroke (width 0) (type default))
+  )
   (wire (pts (xy 189.23 40.64) (xy 189.23 78.74))
     (stroke (width 0) (type default))
@@
     (stroke (width 0) (type default))
   )
+  (wire (pts (xy 93.98 66.04) (xy 93.98 48.26))
+    (stroke (width 0) (type default))
+  )
   (wire (pts (xy 76.2 76.2) (xy 152.4 76.2))
     (stroke (width 0) (type default))
   )
-  (wire (pts (xy 76.2 48.26) (xy 104.14 48.26))
+  (wire (pts (xy 87.63 63.5) (xy 87.63 45.72))
+    (stroke (width 0) (type default))
+  )
+  (wire (pts (xy 76.2 48.26) (xy 93.98 48.26))
     (stroke (width 0) (type default))
   )
@@
       )
     )
+  )
+  (sheet (at 104.14 60.96) (size 17.78 11.43) (fields_autoplaced)
+    (stroke (width 0.1524) (type solid))
+    (fill (color 0 0 0 0.0000))
+    (property "Sheetname" "ACC" (at 104.14 60.2484 0)
+      (effects (font (size 1.27 1.27)) (justify left bottom))
+    )
+    (property "Sheetfile" "acc.kicad_sch" (at 104.14 72.9746 0)
+      (effects (font (size 1.27 1.27)) (justify left top))
+    )
+    (pin "SDA" bidirectional (at 104.14 66.04 180)
+      (effects (font (size 1.27 1.27)) (justify left))
+    )
+    (pin "SCL" input (at 104.14 63.5 180)
+      (effects (font (size 1.27 1.27)) (justify left))
+    )
+    (instances
+      (project "Xaar128-Driver"
+        (path "/f0c82013-03f9-4093-aa02-30b89fd69529" (page "10"))
+      )
+    )
