File: Xaar128-Driver/acc.kicad_sch (KiCad schematic)
At the start: 13 parts, among them U22 LIS2DH

Commit message: create order list
Parts:
- JP16: RSBestNr 120-432 -> (none); Supplier RS -> None
Changed lines of the file:
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@@
       (effects (font (size 1.27 1.27)) hide)
     )
-    (property "RSBestNr" "120-432" (at 48.26 73.66 0)
-      (effects (font (size 1.27 1.27)) hide)
-    )
-    (property "Supplier" "RS" (at 48.26 73.66 0)
+    (property "RSBestNr" "" (at 48.26 73.66 0)
+      (effects (font (size 1.27 1.27)) hide)
+    )
+    (property "Supplier" "None" (at 48.26 73.66 0)
       (effects (font (size 1.27 1.27)) hide)
     )
@@
       (effects (font (size 1.27 1.27)) hide)
     )
-    (property "RSBestNr" "120-432" (at 100.33 102.87 0)
-      (effects (font (size 1.27 1.27)) hide)
-    )
-    (property "Supplier" "RS" (at 100.33 102.87 0)
+    (property "RSBestNr" "" (at 100.33 102.87 0)
+      (effects (font (size 1.27 1.27)) hide)
+    )
+    (property "Supplier" "None" (at 100.33 102.87 0)
       (effects (font (size 1.27 1.27)) hide)
     )
@@
       (effects (font (size 1.27 1.27)) hide)
     )
-    (property "RSBestNr" "120-432" (at 95.25 44.45 0)
-      (effects (font (size 1.27 1.27)) hide)
-    )
-    (property "Supplier" "RS" (at 95.25 44.45 0)
+    (property "RSBestNr" "" (at 95.25 44.45 0)
+      (effects (font (size 1.27 1.27)) hide)
+    )
+    (property "Supplier" "None" (at 95.25 44.45 0)
       (effects (font (size 1.27 1.27)) hide)
     )
@@
       (effects (font (size 1.27 1.27)) hide)
     )
-    (property "RSBestNr" "120-432" (at 48.26 77.47 0)
-      (effects (font (size 1.27 1.27)) hide)
-    )
-    (property "Supplier" "RS" (at 48.26 77.47 0)
-      (effects (font (size 1.27 1.27)) hide)
-    )
+    (property "RSBestNr" "" (at 48.26 77.47 0)
+      (effects (font (size 1.27 1.27)) hide)
+    )
+    (property "Supplier" "None" (at 48.26 77.47 0)
+      (effects (font (size 1.27 1.27)) hide)
+    )

Commit message: fix dac address r
Parts:
- renumbered C21 to C33, JP16 to JP17, JP16 to JP18, JP16 to JP19, JP16 to JP20, NT3 to NT2, NT3 to NT5, R17 to R47, R17 to R48, R17 to R53, TP1 to TP14, TP1 to TP15
