File: Xaar128-Driver/printhead_connector.kicad_sch (KiCad schematic)
At the start: 2 parts, among them J5 Conn_01x21, J6 Conn_02x08_Odd_Even

Commit message: assign footprints
Parts:
- J5: footprint (none) -> Molex_200528:Molex_200528-0210_1x21-1MP_P1.00mm_Horizontal; Supplier (none) -> Printerbox
- J6: footprint (none) -> Connector_IDC:IDC-Header_2x08_P2.54mm_Vertical; RSBestNr (none) -> 771-8357; Supplier (none) -> RS; now not fitted
Changed lines of the file:
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@@
   )
   (symbol (lib_id "Connector_Generic:Conn_02x08_Odd_Even") (at 124.46 105.41 0) (unit 1)
-    (in_bom yes) (on_board yes) (dnp no) (fields_autoplaced)
+    (in_bom yes) (on_board yes) (dnp yes) (fields_autoplaced)
     (property "Reference" "J6" (at 125.73 91.44 0)
       (effects (font (size 1.27 1.27)))
@@
       (effects (font (size 1.27 1.27)))
     )
-    (property "Footprint" "" (at 124.46 105.41 0)
+    (property "Footprint" "Connector_IDC:IDC-Header_2x08_P2.54mm_Vertical" (at 124.46 105.41 0)
       (effects (font (size 1.27 1.27)) hide)
     )
@@
       (effects (font (size 1.27 1.27)) hide)
     )
-    (property "RSBestNr" "" (at 124.46 105.41 0)
-      (effects (font (size 1.27 1.27)) hide)
-    )
-    (property "Supplier" "" (at 124.46 105.41 0)
+    (property "RSBestNr" "771-8357" (at 124.46 105.41 0)
+      (effects (font (size 1.27 1.27)) hide)
+    )
+    (property "Supplier" "RS" (at 124.46 105.41 0)
       (effects (font (size 1.27 1.27)) hide)
     )
@@
       (effects (font (size 1.27 1.27)) (justify left) hide)
     )
-    (property "Footprint" "" (at 162.56 100.33 0)
+    (property "Footprint" "Molex_200528:Molex_200528-0210_1x21-1MP_P1.00mm_Horizontal" (at 162.56 100.33 0)
       (effects (font (size 1.27 1.27)) hide)
     )
@@
       (effects (font (size 1.27 1.27)) hide)
     )
-    (property "Supplier" "" (at 162.56 100.33 0)
-      (effects (font (size 1.27 1.27)) hide)
-    )
+    (property "Supplier" "Printerbox" (at 162.56 100.33 0)
+      (effects (font (size 1.27 1.27)) hide)
+    )

Commit message: xaar driver: some routed islands
Connections:
- net GNDHP renamed GND1
Changed lines of the file:
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@@
     (effects (font (size 1.27 1.27)) (justify right))
   )
-  (symbol (lib_id "Xaar_Driver:GNDHP") (at 154.94 82.55 270) (unit 1)
-    (in_bom yes) (on_board yes) (dnp no) (fields_autoplaced)
-    (property "Reference" "#PWR091" (at 148.59 82.55 0)
-      (effects (font (size 1.27 1.27)) hide)
-    )
-    (property "Value" "GNDHP" (at 151.13 82.55 90)
+  (symbol (lib_id "power:GND1") (at 154.94 82.55 270) (unit 1)
+    (in_bom yes) (on_board yes) (dnp no) (fields_autoplaced)
+    (property "Reference" "#PWR0117" (at 148.59 82.55 0)
+      (effects (font (size 1.27 1.27)) hide)
+    )
+    (property "Value" "GND1" (at 151.13 82.55 90)
       (effects (font (size 1.27 1.27)) (justify right))
     )
@@
       (project "Xaar128-Driver"
         (path "/f0c82013-03f9-4093-aa02-30b89fd69529/00d9c6da-e931-4ba1-a353-d1b49c742a57"
-          (reference "#PWR091") (unit 1)
+          (reference "#PWR0117") (unit 1)
         )
       )
@@
     )
   )
-  (symbol (lib_id "Xaar_Driver:GNDHP") (at 116.84 102.87 270) (unit 1)
-    (in_bom yes) (on_board yes) (dnp no) (fields_autoplaced)
-    (property "Reference" "#PWR094" (at 110.49 102.87 0)
-      (effects (font (size 1.27 1.27)) hide)
-    )
-    (property "Value" "GNDHP" (at 113.03 102.87 90)
+  (symbol (lib_id "power:GND1") (at 116.84 102.87 270) (unit 1)
+    (in_bom yes) (on_board yes) (dnp no) (fields_autoplaced)
+    (property "Reference" "#PWR0115" (at 110.49 102.87 0)
+      (effects (font (size 1.27 1.27)) hide)
+    )
+    (property "Value" "GND1" (at 113.03 102.87 90)
       (effects (font (size 1.27 1.27)) (justify right))
     )
@@
       (project "Xaar128-Driver"
         (path "/f0c82013-03f9-4093-aa02-30b89fd69529/00d9c6da-e931-4ba1-a353-d1b49c742a57"
-          (reference "#PWR094") (unit 1)
-        )
-      )
-    )
-  )
-  (symbol (lib_id "Xaar_Driver:GNDHP") (at 134.62 97.79 90) (unit 1)
-    (in_bom yes) (on_board yes) (dnp no) (fields_autoplaced)
-    (property "Reference" "#PWR081" (at 140.97 97.79 0)
-      (effects (font (size 1.27 1.27)) hide)
-    )
-    (property "Value" "GNDHP" (at 138.43 97.79 90)
+          (reference "#PWR0115") (unit 1)
+        )
+      )
+    )
+  )
+  (symbol (lib_id "power:GND1") (at 134.62 97.79 90) (unit 1)
+    (in_bom yes) (on_board yes) (dnp no) (fields_autoplaced)
+    (property "Reference" "#PWR0114" (at 140.97 97.79 0)
+      (effects (font (size 1.27 1.27)) hide)
+    )
+    (property "Value" "GND1" (at 138.43 97.79 90)
       (effects (font (size 1.27 1.27)) (justify right))
     )
@@
       (project "Xaar128-Driver"
         (path "/f0c82013-03f9-4093-aa02-30b89fd69529/00d9c6da-e931-4ba1-a353-d1b49c742a57"
-          (reference "#PWR081") (unit 1)
+          (reference "#PWR0114") (unit 1)
         )
       )
@@
     )
   )
-  (symbol (lib_id "Xaar_Driver:GNDHP") (at 154.94 77.47 270) (unit 1)
-    (in_bom yes) (on_board yes) (dnp no) (fields_autoplaced)
-    (property "Reference" "#PWR046" (at 148.59 77.47 0)
-      (effects (font (size 1.27 1.27)) hide)
-    )
-    (property "Value" "GNDHP" (at 151.13 77.47 90)
+  (symbol (lib_id "power:GND1") (at 154.94 77.47 270) (unit 1)
+    (in_bom yes) (on_board yes) (dnp no) (fields_autoplaced)
+    (property "Reference" "#PWR0116" (at 148.59 77.47 0)
+      (effects (font (size 1.27 1.27)) hide)
+    )
+    (property "Value" "GND1" (at 151.13 77.47 90)
       (effects (font (size 1.27 1.27)) (justify right))
     )
@@
       (project "Xaar128-Driver"
         (path "/f0c82013-03f9-4093-aa02-30b89fd69529/00d9c6da-e931-4ba1-a353-d1b49c742a57"
-          (reference "#PWR046") (unit 1)
-        )
-      )
+          (reference "#PWR0116") (unit 1)
+        )
+      )
