File: Xaar128-Driver/strobe.kicad_sch (KiCad schematic)
At the start: 6 parts, among them Q3 DMN2075U

Commit message: some component selections, fix wrong mcu
Parts:
- C1: value 100n -> 100n >16V Film; footprint Capacitor_THT:C_Rect_L7.0mm_W2.0mm_P5.00mm -> (none)
- NT2, NT6, NT7: footprint (none) -> NetTie:NetTie-2_SMD_Pad0.5mm; Supplier (none) -> None
- Q3: RSBestNr (none) -> 751-4143; Supplier (none) -> RS
- R2: footprint Resistor_THT:R_Axial_DIN0207_L6.3mm_D2.5mm_P7.62mm_Horizontal -> (none)
Changed lines of the file:
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@@
       (effects (font (size 1.27 1.27)) hide)
     )
-    (property "Footprint" "" (at 140.97 118.11 0)
+    (property "Footprint" "NetTie:NetTie-2_SMD_Pad0.5mm" (at 140.97 118.11 0)
       (effects (font (size 1.27 1.27)) hide)
     )
     (property "Datasheet" "~" (at 140.97 118.11 0)
+      (effects (font (size 1.27 1.27)) hide)
+    )
+    (property "RSBestNr" "" (at 140.97 118.11 0)
+      (effects (font (size 1.27 1.27)) hide)
+    )
+    (property "Supplier" "None" (at 140.97 118.11 0)
       (effects (font (size 1.27 1.27)) hide)
     )
@@
       (effects (font (size 1.27 1.27)))
     )
-    (property "Value" "100n" (at 125.73 100.33 90)
+    (property "Value" "100n >16V Film" (at 125.73 100.33 90)
       (effects (font (size 1.27 1.27)))
     )
-    (property "Footprint" "Capacitor_THT:C_Rect_L7.0mm_W2.0mm_P5.00mm" (at 129.54 104.4448 0)
+    (property "Footprint" "" (at 129.54 104.4448 0)
       (effects (font (size 1.27 1.27)) hide)
     )
     (property "Datasheet" "~" (at 125.73 105.41 0)
+      (effects (font (size 1.27 1.27)) hide)
+    )
+    (property "RSBestNr" "" (at 125.73 105.41 0)
+      (effects (font (size 1.27 1.27)) hide)
+    )
+    (property "Supplier" "" (at 125.73 105.41 0)
       (effects (font (size 1.27 1.27)) hide)
     )
@@
       (effects (font (size 1.27 1.27)) (justify left))
     )
-    (property "Footprint" "Resistor_THT:R_Axial_DIN0207_L6.3mm_D2.5mm_P7.62mm_Horizontal" (at 134.112 110.49 90)
+    (property "Footprint" "" (at 134.112 110.49 90)
       (effects (font (size 1.27 1.27)) hide)
     )
     (property "Datasheet" "~" (at 135.89 110.49 0)
+      (effects (font (size 1.27 1.27)) hide)
+    )
+    (property "RSBestNr" "" (at 135.89 110.49 0)
+      (effects (font (size 1.27 1.27)) hide)
+    )
+    (property "Supplier" "" (at 135.89 110.49 0)
       (effects (font (size 1.27 1.27)) hide)
     )
@@
       (effects (font (size 1.27 1.27)) (justify left) hide)
     )
+    (property "RSBestNr" "751-4143" (at 148.59 100.33 0)
+      (effects (font (size 1.27 1.27)) hide)
+    )
+    (property "Supplier" "RS" (at 148.59 100.33 0)
+      (effects (font (size 1.27 1.27)) hide)
+    )
     (pin "1")
     (pin "2")
@@
       (effects (font (size 1.27 1.27)) hide)
     )
-    (property "Footprint" "" (at 157.48 121.92 0)
+    (property "Footprint" "NetTie:NetTie-2_SMD_Pad0.5mm" (at 157.48 121.92 0)
       (effects (font (size 1.27 1.27)) hide)
     )
     (property "Datasheet" "~" (at 157.48 121.92 0)
+      (effects (font (size 1.27 1.27)) hide)
+    )
+    (property "RSBestNr" "" (at 157.48 121.92 0)
+      (effects (font (size 1.27 1.27)) hide)
+    )
+    (property "Supplier" "None" (at 157.48 121.92 0)
       (effects (font (size 1.27 1.27)) hide)
     )
@@
       (effects (font (size 1.27 1.27)) hide)
     )
-    (property "Footprint" "" (at 147.32 78.74 0)
+    (property "Footprint" "NetTie:NetTie-2_SMD_Pad0.5mm" (at 147.32 78.74 0)
       (effects (font (size 1.27 1.27)) hide)
     )
@@
       (effects (font (size 1.27 1.27)) hide)
     )
+    (property "RSBestNr" "" (at 147.32 78.74 0)
+      (effects (font (size 1.27 1.27)) hide)
+    )
+    (property "Supplier" "None" (at 147.32 78.74 0)
+      (effects (font (size 1.27 1.27)) hide)
+    )

Commit message: assign footprints
Parts:
- C1: footprint (none) -> Capacitor_THT:C_Rect_L7.0mm_W3.5mm_P5.00mm; RSBestNr (none) -> 463-1765; Supplier (none) -> RS
- R2: value 10K -> 10k; footprint (none) -> Resistor_SMD:R_0603_1608Metric_Pad0.98x0.95mm_HandSolder; Supplier (none) -> Elektroplatz
Changed lines of the file:
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@@
       (effects (font (size 1.27 1.27)))
     )
-    (property "Footprint" "" (at 129.54 104.4448 0)
+    (property "Footprint" "Capacitor_THT:C_Rect_L7.0mm_W3.5mm_P5.00mm" (at 129.54 104.4448 0)
       (effects (font (size 1.27 1.27)) hide)
     )
@@
       (effects (font (size 1.27 1.27)) hide)
     )
-    (property "RSBestNr" "" (at 125.73 105.41 0)
+    (property "RSBestNr" "463-1765" (at 125.73 105.41 0)
       (effects (font (size 1.27 1.27)) hide)
     )
-    (property "Supplier" "" (at 125.73 105.41 0)
+    (property "Supplier" "RS" (at 125.73 105.41 0)
       (effects (font (size 1.27 1.27)) hide)
     )
@@
       (effects (font (size 1.27 1.27)) (justify left))
     )
-    (property "Value" "10K" (at 138.43 111.76 0)
+    (property "Value" "10k" (at 138.43 111.76 0)
       (effects (font (size 1.27 1.27)) (justify left))
     )
-    (property "Footprint" "" (at 134.112 110.49 90)
+    (property "Footprint" "Resistor_SMD:R_0603_1608Metric_Pad0.98x0.95mm_HandSolder" (at 134.112 110.49 90)
       (effects (font (size 1.27 1.27)) hide)
     )
@@
       (effects (font (size 1.27 1.27)) hide)
     )
-    (property "Supplier" "" (at 135.89 110.49 0)
+    (property "Supplier" "Elektroplatz" (at 135.89 110.49 0)
       (effects (font (size 1.27 1.27)) hide)
     )

Commit message: more routing
Parts:
- removed NT2, NT6: NetTie_2, NetTie:NetTie-2_SMD_Pad0.5mm, symbol Device:NetTie_2
Connections:
- net LEDPWRGND is gone; now on net GND: Q3.2 (S)
- net GND: now also R2.2
Changed lines of the file:
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@@
     (rev "1.0.0")
   )
-  (junction (at 151.13 121.92) (diameter 0) (color 0 0 0 0)
-  )
   (junction (at 135.89 105.41) (diameter 0) (color 0 0 0 0)
   )
-  (junction (at 151.13 118.11) (diameter 0) (color 0 0 0 0)
-  )
-  (wire (pts (xy 135.89 118.11) (xy 138.43 118.11))
-    (stroke (width 0) (type default))
-  )
   (wire (pts (xy 149.86 78.74) (xy 151.13 78.74))
     (stroke (width 0) (type default))
@@
     (stroke (width 0) (type default))
   )
-  (wire (pts (xy 151.13 105.41) (xy 151.13 118.11))
-    (stroke (width 0) (type default))
-  )
-  (wire (pts (xy 151.13 121.92) (xy 151.13 125.73))
+  (wire (pts (xy 151.13 105.41) (xy 151.13 121.92))
     (stroke (width 0) (type default))
   )
@@
     (stroke (width 0) (type default))
   )
-  (wire (pts (xy 160.02 121.92) (xy 162.56 121.92))
-    (stroke (width 0) (type default))
-  )
-  (wire (pts (xy 151.13 118.11) (xy 151.13 121.92))
+  (wire (pts (xy 151.13 121.92) (xy 162.56 121.92))
     (stroke (width 0) (type default))
   )
@@
     (stroke (width 0) (type default))
   )
-  (wire (pts (xy 154.94 121.92) (xy 151.13 121.92))
-    (stroke (width 0) (type default))
-  )
-  (wire (pts (xy 143.51 118.11) (xy 151.13 118.11))
-    (stroke (width 0) (type default))
-  )
   (wire (pts (xy 115.57 105.41) (xy 121.92 105.41))
     (stroke (width 0) (type default))
@@
   (wire (pts (xy 129.54 105.41) (xy 135.89 105.41))
     (stroke (width 0) (type default))
-  )
-  (global_label "LEDPWRGND" (shape input) (at 151.13 125.73 270) (fields_autoplaced)
-    (effects (font (size 1.27 1.27)) (justify right))
-    (property "Intersheetrefs" "${INTERSHEET_REFS}" (at 151.13 140.0242 90)
-      (effects (font (size 1.27 1.27)) (justify right) hide)
-    )
   )
   (hierarchical_label "LED_PWR" (shape input) (at 143.51 76.2 90) (fields_autoplaced)
@@
     )
   )
-  (netclass_flag "" (length 2.54) (shape round) (at 151.13 124.46 90) (fields_autoplaced)
-    (effects (font (size 1.27 1.27)) (justify left bottom))
-    (property "Netclass" "HP" (at 148.59 123.7615 90)
-      (effects (font (size 1.27 1.27) italic) (justify left))
-    )
-  )
-  (symbol (lib_id "Device:NetTie_2") (at 140.97 118.11 0) (unit 1)
-    (in_bom no) (on_board yes) (dnp no) (fields_autoplaced)
-    (property "Reference" "NT6" (at 140.97 113.03 0)
-      (effects (font (size 1.27 1.27)) hide)
-    )
-    (property "Value" "NetTie_2" (at 140.97 115.57 0)
-      (effects (font (size 1.27 1.27)) hide)
-    )
-    (property "Footprint" "NetTie:NetTie-2_SMD_Pad0.5mm" (at 140.97 118.11 0)
-      (effects (font (size 1.27 1.27)) hide)
-    )
-    (property "Datasheet" "~" (at 140.97 118.11 0)
-      (effects (font (size 1.27 1.27)) hide)
-    )
-    (property "RSBestNr" "" (at 140.97 118.11 0)
-      (effects (font (size 1.27 1.27)) hide)
-    )
-    (property "Supplier" "None" (at 140.97 118.11 0)
-      (effects (font (size 1.27 1.27)) hide)
-    )
-    (pin "1")
-    (pin "2")
-    (instances
-      (project "Xaar128-Driver"
-        (path "/f0c82013-03f9-4093-aa02-30b89fd69529/d69e07d5-2f9c-4e83-9c1b-3f660b6a4d08"
-          (reference "NT6") (unit 1)
-        )
-      )
-    )
-  )
   (symbol (lib_id "Device:C") (at 125.73 105.41 90) (unit 1)
     (in_bom yes) (on_board yes) (dnp no) (fields_autoplaced)
@@
     )
   )
-  (symbol (lib_id "Device:NetTie_2") (at 157.48 121.92 0) (unit 1)
-    (in_bom no) (on_board yes) (dnp no) (fields_autoplaced)
-    (property "Reference" "NT2" (at 157.48 116.84 0)
-      (effects (font (size 1.27 1.27)) hide)
-    )
-    (property "Value" "NetTie_2" (at 157.48 119.38 0)
-      (effects (font (size 1.27 1.27)) hide)
-    )
-    (property "Footprint" "NetTie:NetTie-2_SMD_Pad0.5mm" (at 157.48 121.92 0)
-      (effects (font (size 1.27 1.27)) hide)
-    )
-    (property "Datasheet" "~" (at 157.48 121.92 0)
-      (effects (font (size 1.27 1.27)) hide)
-    )
-    (property "RSBestNr" "" (at 157.48 121.92 0)
-      (effects (font (size 1.27 1.27)) hide)
-    )
-    (property "Supplier" "None" (at 157.48 121.92 0)
-      (effects (font (size 1.27 1.27)) hide)
-    )
-    (pin "1")
-    (pin "2")
-    (instances
-      (project "Xaar128-Driver"
-        (path "/f0c82013-03f9-4093-aa02-30b89fd69529/d69e07d5-2f9c-4e83-9c1b-3f660b6a4d08"
-          (reference "NT2") (unit 1)
-        )
-      )
+  (symbol (lib_id "power:GND") (at 135.89 118.11 0) (unit 1)
+    (in_bom yes) (on_board yes) (dnp no) (fields_autoplaced)
+    (property "Reference" "#PWR063" (at 135.89 124.46 0)
+      (effects (font (size 1.27 1.27)) hide)
+    )
+    (property "Value" "GND" (at 135.89 123.19 0)
+      (effects (font (size 1.27 1.27)))
+    )
+    (property "Footprint" "" (at 135.89 118.11 0)
+      (effects (font (size 1.27 1.27)) hide)
+    )
+    (property "Datasheet" "" (at 135.89 118.11 0)
+      (effects (font (size 1.27 1.27)) hide)
+    )
+    (pin "1")
+    (instances
+      (project "Xaar128-Driver"
+        (path "/f0c82013-03f9-4093-aa02-30b89fd69529/d69e07d5-2f9c-4e83-9c1b-3f660b6a4d08"
+          (reference "#PWR063") (unit 1)
+        )
+      )

Commit message: fix dac address r
Parts:
- renumbered Q3 to Q9
