File: Xaar128-Adapter/Xaar128-Adapter.kicad_pcb (KiCad board)
At the start: 2 copper layers, 41 x 38 mm, 15 parts, among them J1 Conn_01x21, J2 Conn_02x15_Odd_Even, J3 Conn_01x12, Q1 DMN2075U

Commit message: create order list
Parts:
- R6: value 3k-6.8k -> 5.1k > 300mW; footprint Resistor_SMD:R_1210_3225Metric_Pad1.30x2.65mm_HandSolder -> Resistor_SMD:R_0805_2012Metric_Pad1.20x1.40mm_HandSolder
Changed lines of the file:
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@@
     (property "Sheetfile" "Xaar128-Adapter.kicad_sch")
     (property "Sheetname" "")
+    (property "Supplier" "None")
     (property "ki_description" "Mounting Hole without connection")
     (property "ki_keywords" "mounting hole")
@@
     (property "Sheetfile" "Xaar128-Adapter.kicad_sch")
     (property "Sheetname" "")
+    (property "Supplier" "None")
     (property "ki_description" "Mounting Hole without connection")
     (property "ki_keywords" "mounting hole")
@@
     (property "Sheetfile" "Xaar128-Adapter.kicad_sch")
     (property "Sheetname" "")
+    (property "Supplier" "None")
     (property "exclude_from_bom" "")
     (property "ki_description" "Net tie, 2 pins")
@@
     (property "Sheetfile" "Xaar128-Adapter.kicad_sch")
     (property "Sheetname" "")
+    (property "Supplier" "None")
     (property "exclude_from_bom" "")
     (property "ki_description" "Net tie, 2 pins")
@@
       (net 5 "VPPH") (pinfunction "2") (pintype "passive"))
   )
-  (footprint "Resistor_SMD:R_1210_3225Metric_Pad1.30x2.65mm_HandSolder" (layer "B.Cu")
+  (footprint "Resistor_SMD:R_0805_2012Metric_Pad1.20x1.40mm_HandSolder" (layer "B.Cu")
     (at 127 100.838)
-    (descr "Resistor SMD 1210 (3225 Metric), square (rectangular) end terminal, IPC_7351 nominal with elongated pad for handsoldering. (Body size source: IPC-SM-782 page 72, https://www.pcb-3d.com/wordpress/wp-content/uploads/ipc-sm-782a_amendment_1_and_2.pdf), generated with kicad-footprint-generator")
+    (descr "Resistor SMD 0805 (2012 Metric), square (rectangular) end terminal, IPC_7351 nominal with elongated pad for handsoldering. (Body size source: IPC-SM-782 page 72, https://www.pcb-3d.com/wordpress/wp-content/uploads/ipc-sm-782a_amendment_1_and_2.pdf), generated with kicad-footprint-generator")
     (tags "resistor handsolder")
     (property "RSBestNr" "721-8223")
@@
     (property "ki_keywords" "R res resistor")
     (attr smd)
-    (fp_text reference "R6" (at 0 2.28) (layer "B.SilkS")
-        (effects (font (size 1 1) (thickness 0.15)) (justify mirror))
-    )
-    (fp_text value "3k-6.8k" (at 0 -2.28) (layer "B.Fab")
-        (effects (font (size 1 1) (thickness 0.15)) (justify mirror))
-    )
-    (fp_text user "${REFERENCE}" (at 0 0) (layer "B.Fab")
-        (effects (font (size 0.8 0.8) (thickness 0.12)) (justify mirror))
-    )
-    (fp_line (start -0.723737 -1.355) (end 0.723737 -1.355)
-      (stroke (width 0.12) (type solid)) (layer "B.SilkS"))
-    (fp_line (start -0.723737 1.355) (end 0.723737 1.355)
-      (stroke (width 0.12) (type solid)) (layer "B.SilkS"))
-    (fp_line (start -2.45 -1.58) (end -2.45 1.58)
-      (stroke (width 0.05) (type solid)) (layer "B.CrtYd"))
-    (fp_line (start -2.45 1.58) (end 2.45 1.58)
-      (stroke (width 0.05) (type solid)) (layer "B.CrtYd"))
-    (fp_line (start 2.45 -1.58) (end -2.45 -1.58)
-      (stroke (width 0.05) (type solid)) (layer "B.CrtYd"))
-    (fp_line (start 2.45 1.58) (end 2.45 -1.58)
-      (stroke (width 0.05) (type solid)) (layer "B.CrtYd"))
-    (fp_line (start -1.6 -1.245) (end -1.6 1.245)
-      (stroke (width 0.1) (type solid)) (layer "B.Fab"))
-    (fp_line (start -1.6 1.245) (end 1.6 1.245)
-      (stroke (width 0.1) (type solid)) (layer "B.Fab"))
-    (fp_line (start 1.6 -1.245) (end -1.6 -1.245)
-      (stroke (width 0.1) (type solid)) (layer "B.Fab"))
-    (fp_line (start 1.6 1.245) (end 1.6 -1.245)
-      (stroke (width 0.1) (type solid)) (layer "B.Fab"))
-    (pad "1" smd roundrect (at -1.55 0) (size 1.3 2.65) (layers "B.Cu" "B.Paste" "B.Mask") (roundrect_rratio 0.1923076923)
+    (fp_text reference "R6" (at 0 1.65 180) (layer "B.SilkS")
+        (effects (font (size 1 1) (thickness 0.15)) (justify mirror))
+    )
+    (fp_text value "5.1k > 300mW" (at 0 -1.65 180) (layer "B.Fab")
+        (effects (font (size 1 1) (thickness 0.15)) (justify mirror))
+    )
+    (fp_text user "${REFERENCE}" (at 0 0 180) (layer "B.Fab")
+        (effects (font (size 0.5 0.5) (thickness 0.08)) (justify mirror))
+    )
+    (fp_line (start -0.227064 -0.735) (end 0.227064 -0.735)
+      (stroke (width 0.12) (type solid)) (layer "B.SilkS"))
+    (fp_line (start -0.227064 0.735) (end 0.227064 0.735)
+      (stroke (width 0.12) (type solid)) (layer "B.SilkS"))
+    (fp_line (start -1.85 -0.95) (end -1.85 0.95)
+      (stroke (width 0.05) (type solid)) (layer "B.CrtYd"))
+    (fp_line (start -1.85 0.95) (end 1.85 0.95)
+      (stroke (width 0.05) (type solid)) (layer "B.CrtYd"))
+    (fp_line (start 1.85 -0.95) (end -1.85 -0.95)
+      (stroke (width 0.05) (type solid)) (layer "B.CrtYd"))
+    (fp_line (start 1.85 0.95) (end 1.85 -0.95)
+      (stroke (width 0.05) (type solid)) (layer "B.CrtYd"))
+    (fp_line (start -1 -0.625) (end -1 0.625)
+      (stroke (width 0.1) (type solid)) (layer "B.Fab"))
+    (fp_line (start -1 0.625) (end 1 0.625)
+      (stroke (width 0.1) (type solid)) (layer "B.Fab"))
+    (fp_line (start 1 -0.625) (end -1 -0.625)
+      (stroke (width 0.1) (type solid)) (layer "B.Fab"))
+    (fp_line (start 1 0.625) (end 1 -0.625)
+      (stroke (width 0.1) (type solid)) (layer "B.Fab"))
+    (pad "1" smd roundrect (at -1 0) (size 1.2 1.4) (layers "B.Cu" "B.Paste" "B.Mask") (roundrect_rratio 0.208333)
       (net 4 "Net-(D2-A)") (pintype "passive"))
-    (pad "2" smd roundrect (at 1.55 0) (size 1.3 2.65) (layers "B.Cu" "B.Paste" "B.Mask") (roundrect_rratio 0.1923076923)
+    (pad "2" smd roundrect (at 1 0) (size 1.2 1.4) (layers "B.Cu" "B.Paste" "B.Mask") (roundrect_rratio 0.208333)
       (net 34 "Net-(NT1-Pad1)") (pintype "passive"))
-    (model "${KICAD6_3DMODEL_DIR}/Resistor_SMD.3dshapes/R_1210_3225Metric.wrl"
+    (model "${KICAD6_3DMODEL_DIR}/Resistor_SMD.3dshapes/R_0805_2012Metric.wrl"
       (offset (xyz 0 0 0))
       (scale (xyz 1 1 1))
@@
     (property "Sheetname" "")
     (property "Supplier" "RS")
+    (property "dnp" "")
     (property "ki_description" "Generic connector, single row, 01x12, script generated (kicad-library-utils/schlib/autogen/connector/)")
     (property "ki_keywords" "connector")
@@
     (descr "Resistor SMD 0603 (1608 Metric), square (rectangular) end terminal, IPC_7351 nominal with elongated pad for handsoldering. (Body size source: IPC-SM-782 page 72, https://www.pcb-3d.com/wordpress/wp-content/uploads/ipc-sm-782a_amendment_1_and_2.pdf), generated with kicad-footprint-generator")
     (tags "resistor handsolder")
-    (property "RSBestNr" "120-561,181-4452")
+    (property "RSBestNr" "678-9875")
     (property "Sheetfile" "Xaar128-Adapter.kicad_sch")
     (property "Sheetname" "")
@@
     (descr "Resistor SMD 0603 (1608 Metric), square (rectangular) end terminal, IPC_7351 nominal with elongated pad for handsoldering. (Body size source: IPC-SM-782 page 72, https://www.pcb-3d.com/wordpress/wp-content/uploads/ipc-sm-782a_amendment_1_and_2.pdf), generated with kicad-footprint-generator")
     (tags "resistor handsolder")
-    (property "RSBestNr" "120-432")
+    (property "RSBestNr" "820-6736")
     (property "Sheetfile" "Xaar128-Adapter.kicad_sch")
     (property "Sheetname" "")
@@
   (segment (start 131.318 94.488) (end 128.275 97.531) (width 0.25) (layer "B.Cu") (net 3))
   (segment (start 128.275 97.531) (end 128.275 98) (width 0.25) (layer "B.Cu") (net 3))
+  (segment (start 125.735 98) (end 125.735 100.573) (width 0.25) (layer "B.Cu") (net 4))
+  (segment (start 125.735 100.573) (end 126 100.838) (width 0.25) (layer "B.Cu") (net 4))
   (segment (start 125.45 98.285) (end 125.735 98) (width 0.25) (layer "B.Cu") (net 4))
-  (segment (start 125.45 100.838) (end 125.45 98.285) (width 0.25) (layer "B.Cu") (net 4))
   (segment (start 125.704 97.567) (end 125.989 97.282) (width 0.25) (layer "B.Cu") (net 4))
   (segment (start 133.236 100.698) (end 133.096 100.838) (width 0.5) (layer "B.Cu") (net 5))

Commit message: Create plots for fabrication
Parts:
- R4: value 470-680 -> 470
- R6: value 5.1k > 300mW -> 5.1k >300mW
Changed lines of the file:
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@@
     (property "Sheetfile" "Xaar128-Adapter.kicad_sch")
     (property "Sheetname" "")
-    (property "Supplier" "Elekroplatz")
+    (property "Supplier" "Elektroplatz")
     (property "ki_description" "Light emitting diode")
     (property "ki_keywords" "LED diode")
@@
     (property "Sheetfile" "Xaar128-Adapter.kicad_sch")
     (property "Sheetname" "")
-    (property "Supplier" "Elekroplatz")
+    (property "Supplier" "Elektroplatz")
     (property "ki_description" "Light emitting diode")
     (property "ki_keywords" "LED diode")
@@
     (descr "Resistor SMD 0603 (1608 Metric), square (rectangular) end terminal, IPC_7351 nominal with elongated pad for handsoldering. (Body size source: IPC-SM-782 page 72, https://www.pcb-3d.com/wordpress/wp-content/uploads/ipc-sm-782a_amendment_1_and_2.pdf), generated with kicad-footprint-generator")
     (tags "resistor handsolder")
-    (property "RSBestNr" "199-5618")
+    (property "RSBestNr" "566-547")
     (property "Sheetfile" "Xaar128-Adapter.kicad_sch")
     (property "Sheetname" "")
@@
         (effects (font (size 1 1) (thickness 0.15)) (justify mirror))
     )
-    (fp_text value "470-680" (at 0 -1.43 -270) (layer "B.Fab")
+    (fp_text value "470" (at 0 -1.43 -270) (layer "B.Fab")
         (effects (font (size 1 1) (thickness 0.15)) (justify mirror))
     )
@@
     (descr "Resistor SMD 0805 (2012 Metric), square (rectangular) end terminal, IPC_7351 nominal with elongated pad for handsoldering. (Body size source: IPC-SM-782 page 72, https://www.pcb-3d.com/wordpress/wp-content/uploads/ipc-sm-782a_amendment_1_and_2.pdf), generated with kicad-footprint-generator")
     (tags "resistor handsolder")
-    (property "RSBestNr" "721-8223")
+    (property "RSBestNr" "721-7804")
     (property "Sheetfile" "Xaar128-Adapter.kicad_sch")
     (property "Sheetname" "")
@@
         (effects (font (size 1 1) (thickness 0.15)) (justify mirror))
     )
-    (fp_text value "5.1k > 300mW" (at 0 -1.65 180) (layer "B.Fab")
+    (fp_text value "5.1k >300mW" (at 0 -1.65 180) (layer "B.Fab")
         (effects (font (size 1 1) (thickness 0.15)) (justify mirror))
     )
@@
     (fp_line (start 1 0.625) (end 1 -0.625)
       (stroke (width 0.1) (type solid)) (layer "B.Fab"))
-    (pad "1" smd roundrect (at -1 0) (size 1.2 1.4) (layers "B.Cu" "B.Paste" "B.Mask") (roundrect_rratio 0.208333)
+    (pad "1" smd roundrect (at -1 0) (size 1.2 1.4) (layers "B.Cu" "B.Paste" "B.Mask") (roundrect_rratio 0.2083333333)
       (net 4 "Net-(D2-A)") (pintype "passive"))
-    (pad "2" smd roundrect (at 1 0) (size 1.2 1.4) (layers "B.Cu" "B.Paste" "B.Mask") (roundrect_rratio 0.208333)
+    (pad "2" smd roundrect (at 1 0) (size 1.2 1.4) (layers "B.Cu" "B.Paste" "B.Mask") (roundrect_rratio 0.2083333333)
       (net 34 "Net-(NT1-Pad1)") (pintype "passive"))
     (model "${KICAD6_3DMODEL_DIR}/Resistor_SMD.3dshapes/R_0805_2012Metric.wrl"
@@
     (property "Sheetfile" "Xaar128-Adapter.kicad_sch")
     (property "Sheetname" "")
-    (property "Supplier" "Inkjetbox")
+    (property "Supplier" "Printerbox")
     (property "ki_description" "Generic connector, single row, 01x21, script generated (kicad-library-utils/schlib/autogen/connector/)")
     (property "ki_keywords" "connector")
