File: Xaar128-Adapter/Xaar128-Adapter.kicad_sch (KiCad schematic)
At the start: 15 parts, among them J1 Conn_01x21, J2 Conn_02x15_Odd_Even, J3 Conn_01x12, Q1 DMN2075U

Commit message: adapter mostly done
Parts:
- D1, D2: footprint LED_THT:LED_D3.0mm -> Custom_LED_THT:LED_D3.0mm
Changed lines of the file:
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@@
       (effects (font (size 1.27 1.27)) (justify right))
     )
-    (property "Footprint" "LED_THT:LED_D3.0mm" (at 101.6 71.12 0)
+    (property "Footprint" "Custom_LED_THT:LED_D3.0mm" (at 101.6 71.12 0)
       (effects (font (size 1.27 1.27)) hide)
     )
@@
       (effects (font (size 1.27 1.27)) (justify right))
     )
-    (property "Footprint" "LED_THT:LED_D3.0mm" (at 59.69 71.12 0)
-      (effects (font (size 1.27 1.27)) hide)
-    )
+    (property "Footprint" "Custom_LED_THT:LED_D3.0mm" (at 59.69 71.12 0)
+      (effects (font (size 1.27 1.27)) hide)
+    )

Commit message: create order list
Parts:
- D1, D2: Supplier Elekroplatz -> Elektroplatz
- H1, H2, NT1, NT2: Supplier (none) -> None
- J1: Supplier Inkjetbox -> Printerbox
- J3: now not fitted
- R1: RSBestNr 120-432 -> 820-6736
- R3: RSBestNr 120-561,181-4452 -> 678-9875
- R4: value 470-680 -> 470; RSBestNr 199-5618 -> 566-547
- R6: value 3k-6.8k -> 5.1k >300mW; footprint Resistor_SMD:R_1210_3225Metric_Pad1.30x2.65mm_HandSolder -> Resistor_SMD:R_0805_2012Metric_Pad1.20x1.40mm_HandSolder; RSBestNr 721-8223 -> 721-7804
Changed lines of the file:
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@@
       (effects (font (size 1.27 1.27)) hide)
     )
-    (property "RSBestNr" "120-561,181-4452" (at 49.53 80.01 0)
+    (property "RSBestNr" "678-9875" (at 49.53 80.01 0)
       (effects (font (size 1.27 1.27)) hide)
     )
@@
       (effects (font (size 1.27 1.27)) hide)
     )
-    (property "Supplier" "Inkjetbox" (at 265.43 73.66 0)
+    (property "Supplier" "Printerbox" (at 265.43 73.66 0)
       (effects (font (size 1.27 1.27)) hide)
     )
@@
       (effects (font (size 1.27 1.27)) hide)
     )
+    (property "Supplier" "None" (at 59.69 22.86 0)
+      (effects (font (size 1.27 1.27)) hide)
+    )
     (instances
       (project "Xaar128-Adapter"
@@
       (effects (font (size 1.27 1.27)) hide)
     )
-    (property "Supplier" "Elekroplatz" (at 101.6 71.12 0)
+    (property "Supplier" "Elektroplatz" (at 101.6 71.12 0)
       (effects (font (size 1.27 1.27)) hide)
     )
@@
       (effects (font (size 1.27 1.27)) hide)
     )
+    (property "Supplier" "None" (at 101.6 49.53 0)
+      (effects (font (size 1.27 1.27)) hide)
+    )
     (pin "1")
     (pin "2")
@@
   )
   (symbol (lib_id "Connector_Generic:Conn_01x12") (at 231.14 124.46 0) (mirror x) (unit 1)
-    (in_bom yes) (on_board yes) (dnp no)
+    (in_bom yes) (on_board yes) (dnp yes)
     (property "Reference" "J3" (at 233.68 124.46 0)
       (effects (font (size 1.27 1.27)) (justify left))
@@
       (effects (font (size 1.27 1.27)) hide)
     )
+    (property "Supplier" "None" (at 59.69 27.94 0)
+      (effects (font (size 1.27 1.27)) hide)
+    )
     (instances
       (project "Xaar128-Adapter"
@@
       (effects (font (size 1.27 1.27)) hide)
     )
+    (property "Supplier" "None" (at 101.6 88.9 0)
+      (effects (font (size 1.27 1.27)) hide)
+    )
     (pin "1")
     (pin "2")
@@
       (effects (font (size 1.27 1.27)) hide)
     )
-    (property "RSBestNr" "120-432" (at 157.48 115.57 0)
+    (property "RSBestNr" "820-6736" (at 157.48 115.57 0)
       (effects (font (size 1.27 1.27)) hide)
     )
@@
       (effects (font (size 1.27 1.27)) (justify right))
     )
-    (property "Value" "470-680" (at 62.23 60.96 0)
+    (property "Value" "470" (at 62.23 60.96 0)
       (effects (font (size 1.27 1.27)) (justify right))
     )
@@
       (effects (font (size 1.27 1.27)) hide)
     )
-    (property "RSBestNr" "199-5618" (at 59.69 59.69 0)
+    (property "RSBestNr" "566-547" (at 59.69 59.69 0)
       (effects (font (size 1.27 1.27)) hide)
     )
@@
       (effects (font (size 1.27 1.27)) hide)
     )
-    (property "Supplier" "Elekroplatz" (at 59.69 71.12 0)
+    (property "Supplier" "Elektroplatz" (at 59.69 71.12 0)
       (effects (font (size 1.27 1.27)) hide)
     )
@@
       (effects (font (size 1.27 1.27)) (justify right))
     )
-    (property "Value" "3k-6.8k" (at 104.14 60.96 0)
-      (effects (font (size 1.27 1.27)) (justify right))
-    )
-    (property "Footprint" "Resistor_SMD:R_1210_3225Metric_Pad1.30x2.65mm_HandSolder" (at 103.378 59.69 90)
+    (property "Value" "5.1k >300mW" (at 104.14 60.96 0)
+      (effects (font (size 1.27 1.27)) (justify right))
+    )
+    (property "Footprint" "Resistor_SMD:R_0805_2012Metric_Pad1.20x1.40mm_HandSolder" (at 103.378 59.69 90)
       (effects (font (size 1.27 1.27)) hide)
     )
@@
       (effects (font (size 1.27 1.27)) hide)
     )
-    (property "RSBestNr" "721-8223" (at 101.6 59.69 0)
-      (effects (font (size 1.27 1.27)) hide)
-    )
+    (property "RSBestNr" "721-7804" (at 101.6 59.69 0)
+      (effects (font (size 1.27 1.27)) hide)
+    )

Commit message: ordering voltage regulator extension
Parts:
- J2: Supplier RS -> Printerbox
Changed lines of the file:
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@@
       (effects (font (size 1.27 1.27)) hide)
     )
-    (property "Supplier" "RS" (at 194.31 76.2 0)
+    (property "Supplier" "Printerbox" (at 194.31 76.2 0)
       (effects (font (size 1.27 1.27)) hide)
     )
