File: pump/pump.kicad_pcb (KiCad board)
At the start: 2 copper layers, 7 parts, among them J1 Conn_01x08_Socket, J2 Conn_01x08_Socket, J3 Conn_01x04_Socket, J4 Screw_Terminal_01x02, J5 Screw_Terminal_01x02, J6 Conn_01x01_Socket

Commit message: implement pressure control on nucleo
Parts:
- moved J1 3.56 mm to (91.5, 101.6)
- moved J2 3.56 mm to (106.7, 101.6)
- moved J3 3.56 mm to (114.3, 109.2)
- moved J4 3.56 mm to (86.4, 119.4)
- moved J5 3.56 mm to (86.4, 109.2)
- moved J6 3.56 mm to (109.3, 91.4)
- moved R1 3.56 mm to (99.1, 109.2)
Connections:
- J3 pad 1: BIN1 -> GND
- J3 pad 2: GND -> BIN1
Routing:
- net GND: track 59.5 -> 62.0 mm
- net BIN1: track 8.67 -> 7.62 mm
Changed lines of the file:
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@@
   (net 14 "PWMB")
   (footprint "Resistor_THT:R_Axial_DIN0207_L6.3mm_D2.5mm_P7.62mm_Horizontal" (layer "F.Cu")
-    (at 101.6 106.68 90)
+    (at 99.1 109.22 90)
     (descr "Resistor, Axial_DIN0207 series, Axial, Horizontal, pin pitch=7.62mm, 0.25W = 1/4W, length*diameter=6.3*2.5mm^2, http://cdn-reichelt.de/documents/datenblatt/B400/1_4W%23YAG.pdf")
     (tags "Resistor Axial_DIN0207 series Axial Horizontal pin pitch 7.62mm 0.25W = 1/4W length 6.3mm diameter 2.5mm")
@@
   )
   (footprint "Connector_PinSocket_2.54mm:PinSocket_1x08_P2.54mm_Vertical" (layer "F.Cu")
-    (at 109.22 99.06)
+    (at 106.72 101.6)
     (descr "Through hole straight socket strip, 1x08, 2.54mm pitch, single row (from Kicad 4.0.7), script generated")
     (tags "Through hole socket strip THT 1x08 2.54mm single row")
@@
   )
   (footprint "Connector_PinSocket_2.54mm:PinSocket_1x08_P2.54mm_Vertical" (layer "F.Cu")
-    (at 93.98 99.06)
+    (at 91.48 101.6)
     (descr "Through hole straight socket strip, 1x08, 2.54mm pitch, single row (from Kicad 4.0.7), script generated")
     (tags "Through hole socket strip THT 1x08 2.54mm single row")
@@
   )
   (footprint "RS_PRO:Steckbarer_Klemmenblock_1x02_5.08mm_horizontal" (layer "F.Cu")
-    (at 88.9 116.84 90)
+    (at 86.4 119.38 90)
     (descr "simple 2-pin terminal block, pitch 5.08mm, revamped version of bornier2")
     (tags "terminal block bornier2")
@@
   )
   (footprint "RS_PRO:Steckbarer_Klemmenblock_1x02_5.08mm_horizontal" (layer "F.Cu")
-    (at 88.9 106.68 90)
+    (at 86.4 109.22 90)
     (descr "simple 2-pin terminal block, pitch 5.08mm, revamped version of bornier2")
     (tags "terminal block bornier2")
@@
   )
   (footprint "Connector_PinSocket_2.54mm:PinSocket_1x01_P2.54mm_Vertical" (layer "F.Cu")
-    (at 111.76 88.9)
+    (at 109.26 91.44)
     (descr "Through hole straight socket strip, 1x01, 2.54mm pitch, single row (from Kicad 4.0.7), script generated")
     (tags "Through hole socket strip THT 1x01 2.54mm single row")
@@
   )
   (footprint "Connector_PinSocket_2.54mm:PinSocket_1x04_P2.54mm_Vertical" (layer "F.Cu")
-    (at 116.84 106.68)
+    (at 114.34 109.22)
     (descr "Through hole straight socket strip, 1x04, 2.54mm pitch, single row (from Kicad 4.0.7), script generated")
     (tags "Through hole socket strip THT 1x04 2.54mm single row")
@@
       (stroke (width 0.1) (type solid)) (layer "F.Fab"))
     (pad "1" thru_hole rect (at 0 0) (size 1.7 1.7) (drill 1) (layers "*.Cu" "*.Mask")
-      (net 12 "BIN1") (pinfunction "Pin_1") (pintype "passive"))
+      (net 3 "GND") (pinfunction "Pin_1") (pintype "passive"))
     (pad "2" thru_hole oval (at 0 2.54) (size 1.7 1.7) (drill 1) (layers "*.Cu" "*.Mask")
-      (net 3 "GND") (pinfunction "Pin_2") (pintype "passive"))
+      (net 12 "BIN1") (pinfunction "Pin_2") (pintype "passive"))
     (pad "3" thru_hole oval (at 0 5.08) (size 1.7 1.7) (drill 1) (layers "*.Cu" "*.Mask")
       (net 13 "BIN2") (pinfunction "Pin_3") (pintype "passive"))
@@
     )
   )
-  (segment (start 93.98 99.06) (end 91.44 99.06) (width 0.25) (layer "F.Cu") (net 1))
-  (segment (start 91.44 99.06) (end 88.9 101.6) (width 0.25) (layer "F.Cu") (net 1))
-  (segment (start 101.6 101.6) (end 93.98 101.6) (width 0.25) (layer "F.Cu") (net 2))
-  (segment (start 101.6 99.06) (end 101.6 101.6) (width 0.25) (layer "F.Cu") (net 2))
-  (segment (start 93.98 104.14) (end 99.06 104.14) (width 0.25) (layer "F.Cu") (net 3))
-  (segment (start 91.44 104.14) (end 93.98 104.14) (width 0.25) (layer "F.Cu") (net 3))
-  (segment (start 109.22 116.84) (end 119.38 116.84) (width 0.25) (layer "F.Cu") (net 3))
-  (segment (start 99.06 116.84) (end 109.22 116.84) (width 0.25) (layer "F.Cu") (net 3))
-  (segment (start 88.9 106.68) (end 91.44 104.14) (width 0.25) (layer "F.Cu") (net 3))
-  (segment (start 119.38 109.22) (end 116.84 109.22) (width 0.25) (layer "F.Cu") (net 3))
-  (segment (start 119.38 116.84) (end 119.38 109.22) (width 0.25) (layer "F.Cu") (net 3))
-  (segment (start 99.06 104.14) (end 99.06 116.84) (width 0.25) (layer "F.Cu") (net 3))
-  (segment (start 93.98 116.84) (end 99.06 116.84) (width 0.25) (layer "F.Cu") (net 3))
-  (segment (start 101.6 106.68) (end 109.22 106.68) (width 0.25) (layer "F.Cu") (net 4))
-  (segment (start 88.9 111.76) (end 93.98 111.76) (width 0.25) (layer "F.Cu") (net 7))
-  (segment (start 88.9 116.84) (end 91.44 114.3) (width 0.25) (layer "F.Cu") (net 8))
-  (segment (start 91.44 114.3) (end 93.98 114.3) (width 0.25) (layer "F.Cu") (net 8))
-  (segment (start 111.76 109.22) (end 114.3 106.68) (width 0.25) (layer "F.Cu") (net 12))
-  (segment (start 114.3 106.68) (end 116.84 106.68) (width 0.25) (layer "F.Cu") (net 12))
-  (segment (start 109.22 109.22) (end 111.76 109.22) (width 0.25) (layer "F.Cu") (net 12))
-  (segment (start 116.84 111.76) (end 109.22 111.76) (width 0.25) (layer "F.Cu") (net 13))
-  (segment (start 116.84 114.3) (end 109.22 114.3) (width 0.25) (layer "F.Cu") (net 14))
+  (segment (start 91.48 101.6) (end 88.94 101.6) (width 0.25) (layer "F.Cu") (net 1))
+  (segment (start 88.94 101.6) (end 86.4 104.14) (width 0.25) (layer "F.Cu") (net 1))
+  (segment (start 99.1 104.14) (end 91.48 104.14) (width 0.25) (layer "F.Cu") (net 2))
+  (segment (start 99.1 101.6) (end 99.1 104.14) (width 0.25) (layer "F.Cu") (net 2))
+  (segment (start 91.48 106.68) (end 96.56 106.68) (width 0.25) (layer "F.Cu") (net 3))
+  (segment (start 88.94 106.68) (end 91.48 106.68) (width 0.25) (layer "F.Cu") (net 3))
+  (segment (start 96.56 119.38) (end 106.72 119.38) (width 0.25) (layer "F.Cu") (net 3))
+  (segment (start 86.4 109.22) (end 88.94 106.68) (width 0.25) (layer "F.Cu") (net 3))
+  (segment (start 96.56 106.68) (end 96.56 119.38) (width 0.25) (layer "F.Cu") (net 3))
+  (segment (start 116.88 109.22) (end 116.88 119.38) (width 0.25) (layer "F.Cu") (net 3))
+  (segment (start 91.48 119.38) (end 96.56 119.38) (width 0.25) (layer "F.Cu") (net 3))
+  (segment (start 116.88 119.38) (end 106.72 119.38) (width 0.25) (layer "F.Cu") (net 3))
+  (segment (start 114.34 109.22) (end 116.88 109.22) (width 0.25) (layer "F.Cu") (net 3))
+  (segment (start 99.1 109.22) (end 106.72 109.22) (width 0.25) (layer "F.Cu") (net 4))
+  (segment (start 86.4 114.3) (end 91.48 114.3) (width 0.25) (layer "F.Cu") (net 7))
+  (segment (start 86.4 119.38) (end 88.94 116.84) (width 0.25) (layer "F.Cu") (net 8))
+  (segment (start 88.94 116.84) (end 91.48 116.84) (width 0.25) (layer "F.Cu") (net 8))
+  (segment (start 114.34 111.76) (end 106.72 111.76) (width 0.25) (layer "F.Cu") (net 12))
+  (segment (start 114.34 114.3) (end 106.72 114.3) (width 0.25) (layer "F.Cu") (net 13))
+  (segment (start 114.34 116.84) (end 106.72 116.84) (width 0.25) (layer "F.Cu") (net 14))
 )

Commit message: wip
Parts:
- added J7: Screw_Terminal_01x02, RS_PRO:Steckbarer_Klemmenblock_1x02_5.08mm_horizontal, F.Cu at (114.2, 105.6)
- moved J6 41.5 mm to (86.2, 125.9), turned to 180 degrees
- moved J4 38.4 mm to (114.2, 92.9), turned to -90 degrees
- moved J3 33.2 mm to (81.1, 108.1), turned to 180 degrees
- moved J5 29.2 mm to (114.2, 118.3), turned to -90 degrees
- moved J2 22.9 mm to (88.7, 115.8), turned to 180 degrees
- moved J1 18.9 mm to (104.0, 115.8), turned to 180 degrees
- moved R1 2.95 mm to (96.4, 108.1), turned to -90 degrees
Connections:
- J1 pad 4: unconnected-(J1-Pin_4-Pad4) -> A01
- J1 pad 5: unconnected-(J1-Pin_5-Pad5) -> A02
- J2 pad 1: unconnected-(J2-Pin_1-Pad1) -> PWMA
- J2 pad 2: unconnected-(J2-Pin_2-Pad2) -> AIN2
- J2 pad 3: unconnected-(J2-Pin_3-Pad3) -> AIN1
Routing:
- net A01: track 0.00 -> 11.3 mm
- net A02: track 0.00 -> 10.2 mm
- net GND: track 62.0 -> 69.2 mm
- net B01: track 6.13 -> 13.4 mm
- net B02: track 5.08 -> 12.3 mm
- net +5V: track 6.13 -> 13.4 mm

Commit message: perfboard supports two pumps
Parts:
- added J8: Conn_01x04_Socket, Connector_PinSocket_2.54mm:PinSocket_1x04_P2.54mm_Vertical, F.Cu at (119.4, 96.5)
- moved J4 45.6 mm to (81.3, 124.5), turned to 90 degrees
- moved J3 38.4 mm to (119.4, 111.8), turned to 0 degrees
- moved J5 38.1 mm to (81.3, 99.1), turned to 90 degrees
- moved J7 33.5 mm to (81.3, 111.8), turned to 90 degrees
- moved J6 33.2 mm to (119.4, 127.0), turned to 0 degrees
- moved J2 22.9 mm to (106.7, 101.6), turned to 0 degrees
- moved J1 18.9 mm to (91.5, 101.6), turned to 0 degrees
- moved R1 2.95 mm to (99.1, 109.2), turned to 90 degrees
Routing:
- net +3.3V: track 10.2 -> 55.8 mm, vias 0 -> 2
- net PWMA: track 0.00 -> 17.8 mm
- net AIN2: track 0.00 -> 15.2 mm
- net AIN1: track 0.00 -> 15.2 mm
- net BIN2: track 7.62 -> 15.2 mm
- net PWMB: track 7.62 -> 15.2 mm
- net BIN1: track 7.62 -> 15.2 mm
- net GND: track 69.2 -> 76.3 mm, vias 0 -> 2
- net B01: track 13.4 -> 17.8 mm
- net +5V: track 13.4 -> 17.8 mm
- net B02: track 12.3 -> 15.3 mm
- net A01: track 11.3 -> 12.7 mm

Commit message: perfboard with second pump
Parts:
- added J9: Conn_01x01_Socket, Connector_PinSocket_2.54mm:PinSocket_1x01_P2.54mm_Vertical, F.Cu at (114.3, 129.5)
- moved J3 5.08 mm to (124.5, 111.8)
- moved J6 5.08 mm to (114.3, 127.0)
- moved J8 5.08 mm to (124.5, 96.5)
Routing:
- net PWMB: track 15.2 -> 20.3 mm
- net PWMA: track 17.8 -> 22.9 mm
- net BIN2: track 15.2 -> 20.3 mm
- net BIN1: track 15.2 -> 20.3 mm
- net AIN2: track 15.2 -> 20.3 mm
- net AIN1: track 15.2 -> 20.3 mm
- net GND: track 76.3 -> 81.3 mm
- net +3.3V: track 55.8 -> 53.3 mm
