File: Heatbed/Heatbed.kicad_sch (KiCad schematic)
At the start: 11 parts, among them J1 Conn_01x04, J2 Conn_01x03, J4 Conn_01x02, Q1 IPP060N06N, Q2 BS170

Commit message: final heatbed circuit
Parts:
- removed J1: Conn_01x04, Connector_PinSocket_2.54mm:PinSocket_1x04_P2.54mm_Vertical, symbol Connector_Generic:Conn_01x04
- added D1: D, Diode_THT:D_A-405_P7.62mm_Horizontal, symbol Device:D
- added D2: LED, LED_THT:LED_D3.0mm, symbol Device:LED
- added J1: Conn_01x02, Connector_PinHeader_2.54mm:PinHeader_1x02_P2.54mm_Vertical, symbol Connector_Generic:Conn_01x02
- added R7: 4k, Resistor_THT:R_Axial_DIN0204_L3.6mm_D1.6mm_P5.08mm_Horizontal, symbol Device:R
- R2: value 4.7k -> 7.5k
Connections:
- net +15 is gone; now on net +24: R1.1
- net +24: now also R7.1
- net HB-: now also D2.1 (K)
- net HB_ACTIVE: now also D1.1 (K), J1.1 (Pin_1); no longer R1.2, R2.1, R4.1
- new net: D2.2 (A), R7.2
- new net: D1.2 (A), R1.2, R2.1, R4.1
- no-connect marks 2 -> 1
Other:
- note added: "(28V)"
- note added: "10.28(12)V/GND"
- note added: "GND/12(14)V"
- note removed: "4.79V/GND"
- note removed: "GND/12V"
